File: elec/adm_shield/adm_shield.kicad_pcb (KiCad board)
At the start: 2 copper layers, 43 parts

Commit message: PCB almost finished ?
Parts:
- removed I2C5: CONN_4, PIN_ARRAY_4x1
- added I2C2: CONN_4, PIN_ARRAY_4x1, F.Cu at (233.7, 115.6)
- moved I2C3 23.0 mm to (210.8, 115.6)
- moved I2C4 11.5 mm to (222.2, 119.4), turned to 0 degrees
- moved SERVO_LB0 5.08 mm to (166.4, 170.2), turned to 180 degrees
- moved SERVO_LB1 5.08 mm to (166.4, 175.3), turned to 180 degrees
- moved SERVO_LB2 5.08 mm to (166.4, 180.3), turned to 180 degrees
- moved SERVO_LF0 3.81 mm to (166.4, 96.5), turned to 180 degrees
- moved SERVO_LF1 3.81 mm to (166.4, 91.4), turned to 180 degrees
- moved SERVO_LF2 3.81 mm to (166.4, 86.4), turned to 180 degrees
- moved SERVO_RB0 3.81 mm to (274.3, 170.2)
- moved SERVO_RB1 3.81 mm to (274.3, 175.3)
- moved SERVO_RB2 3.81 mm to (274.3, 180.3)
- moved SERVO_RF0 3.81 mm to (274.3, 96.5)
- moved SERVO_RF1 3.81 mm to (274.3, 91.4)
- moved SERVO_RF2 3.81 mm to (274.3, 86.4)
- moved I2C0 2.54 mm to (210.8, 102.9)
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Connections:
- SHIELD1 pad 43: (no net) -> /LEG_LB/PWM2
- SHIELD1 pad 47: (no net) -> /LEG_LB/PWM0
Routing:
- net /ALIM/POW_5V: track 0.00 -> 521.6 mm
- net /ARDUINO/LOG_5V: track 0.00 -> 193.3 mm
- net /LEG_RB/PWM1: track 0.00 -> 156.0 mm, vias 0 -> 1
- net /LEG_RB/PWM2: track 0.00 -> 152.2 mm, vias 0 -> 3
- net /ARDUINO/SCL: track 0.00 -> 123.9 mm
- net /LEG_RB/PWM0: track 0.00 -> 117.9 mm
- net /ARDUINO/SDA: track 0.00 -> 116.0 mm, vias 0 -> 2
- net /LEG_LF/PWM2: track 0.00 -> 106.3 mm, vias 0 -> 1
- net /LEG_LF/PWM1: track 0.00 -> 99.4 mm
- net /LEG_LF/PWM0: track 0.00 -> 92.5 mm, vias 0 -> 1
- net /LEG_LB/PWM1: track 0.00 -> 81.2 mm
- net /LEG_RF/PWM1: track 0.00 -> 77.7 mm
- net /LEG_LB/PWM2: track 0.00 -> 77.2 mm
- net /LEG_RF/PWM2: track 0.00 -> 73.6 mm
- net /LEG_LB/PWM0: track 0.00 -> 72.9 mm, vias 0 -> 1
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
Commit message: First version PCB.
Connections:
- SHIELD1 pad 5V_4: /ARDUINO/LOG_5V -> (no net)
- SHIELD1 pad 5V_5: /ARDUINO/LOG_5V -> (no net)
Routing:
- net /ALIM/POW_5V: track 521.6 -> 526.7 mm
- net /ARDUINO/LOG_5V: track 193.3 -> 190.7 mm
- added copper zone on B.Cu, net /ALIM/GND
- added copper zone on F.Cu, net /ALIM/GND
Changed lines of the file:
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@@
 (kicad_pcb (version 3) (host pcbnew "(2013-june-11)-stable")
   (general
-    (links 135)
-    (no_connects 50)
-    (area 0 0 0 0)
+    (links 133)
+    (no_connects 0)
+    (area 160.7058 64.786934 279.9842 200.990201)
     (thickness 1.6)
     (drawings 0)
@@
   (net 34 /LEG_RF/PWM1)
   (net 35 /LEG_RF/PWM2)
-  (net 36 N-0000076)
-  (net 37 N-0000077)
-  (net 38 N-0000078)
+  (net 36 N-0000078)
+  (net 37 N-0000079)
+  (net 38 N-0000080)
   (net_class Default "Ceci est la Netclass par défaut"
     (clearance 0.254)
@@
     (add_net /LEG_RF/PWM1)
     (add_net /LEG_RF/PWM2)
-    (add_net N-0000076)
-    (add_net N-0000077)
     (add_net N-0000078)
+    (add_net N-0000079)
+    (add_net N-0000080)
   )
   (module ARDUINO_MEGA_SHIELD (layer F.Cu)
@@
     (pad 5V_4 thru_hole circle (at 93.98 -50.8 270) (size 1.524 1.524) (drill 0.8128)
       (layers *.Cu *.Mask F.SilkS)
-      (net 7 /ARDUINO/LOG_5V)
     )
     (pad 5V_5 thru_hole circle (at 96.52 -50.8 270) (size 1.524 1.524) (drill 0.8128)
       (layers *.Cu *.Mask F.SilkS)
-      (net 7 /ARDUINO/LOG_5V)
     )
     (pad 31 thru_hole circle (at 96.52 -38.1 270) (size 1.524 1.524) (drill 0.8128)
@@
     (pad 1 thru_hole circle (at 3.81 -2.54 180) (size 1.397 1.397) (drill 0.8128)
       (layers *.Cu *.Mask F.SilkS)
-      (net 38 N-0000078)
+      (net 38 N-0000080)
     )
     (pad 2 thru_hole circle (at 3.81 2.54 180) (size 1.397 1.397) (drill 0.8128)
       (layers *.Cu *.Mask F.SilkS)
-      (net 37 N-0000077)
+      (net 37 N-0000079)
     )
     (pad 1 thru_hole circle (at -3.81 -2.54 180) (size 1.397 1.397) (drill 0.8128)
       (layers *.Cu *.Mask F.SilkS)
-      (net 38 N-0000078)
+      (net 38 N-0000080)
     )
     (pad 2 thru_hole circle (at -3.81 2.54 180) (size 1.397 1.397) (drill 0.8128)
       (layers *.Cu *.Mask F.SilkS)
-      (net 37 N-0000077)
+      (net 37 N-0000079)
     )
   )
@@
     (pad 1 thru_hole rect (at -5.08 0 90) (size 1.524 1.524) (drill 1.016)
       (layers *.Cu *.Mask F.SilkS)
-      (net 36 N-0000076)
+      (net 36 N-0000078)
     )
     (pad 2 thru_hole circle (at -2.54 0 90) (size 1.524 1.524) (drill 1.016)
       (layers *.Cu *.Mask F.SilkS)
-      (net 37 N-0000077)
+      (net 37 N-0000079)
     )
     (pad 3 thru_hole circle (at 0 0 90) (size 1.524 1.524) (drill 1.016)
@@
     (pad 2 thru_hole circle (at 0 0) (size 1.524 1.524) (drill 1.016)
       (layers *.Cu *.Mask F.SilkS)
-      (net 38 N-0000078)
+      (net 38 N-0000080)
     )
     (pad 3 thru_hole circle (at 2.54 0) (size 1.524 1.524) (drill 1.016)
@@
     (pad 1 thru_hole rect (at 0 0) (size 1.524 1.524) (drill 1.016)
       (layers *.Cu *.Mask F.SilkS)
-      (net 36 N-0000076)
+      (net 36 N-0000078)
     )
     (model pin_array\pin_1.wrl
@@
     )
   )
+  (segment (start 166.37 180.34) (end 166.37 175.26) (width 0.75) (layer F.Cu) (net 2))
   (segment (start 274.32 91.44) (end 274.32 86.36) (width 1.5) (layer B.Cu) (net 2))
   (segment (start 177.8 99.06) (end 177.8 105.41) (width 1.5) (layer B.Cu) (net 2))
@@
   (segment (start 185.42 133.35) (end 184.15 133.35) (width 0.5) (layer B.Cu) (net 6))
   (segment (start 195.58 143.51) (end 185.42 133.35) (width 0.5) (layer B.Cu) (net 6))
-  (segment (start 181.61 133.35) (end 181.61 129.54) (width 0.75) (layer B.Cu) (net 7) (status C00000))
-  (segment (start 181.61 137.16) (end 181.61 133.35) (width 0.75) (layer B.Cu) (net 7) (status C00000))
-  (segment (start 181.61 140.97) (end 181.61 137.16) (width 0.75) (layer B.Cu) (net 7) (status C00000))
+  (segment (start 181.61 133.35) (end 181.61 129.54) (width 0.75) (layer B.Cu) (net 7))
+  (segment (start 181.61 137.16) (end 181.61 133.35) (width 0.75) (layer B.Cu) (net 7))
+  (segment (start 181.61 140.97) (end 181.61 137.16) (width 0.75) (layer B.Cu) (net 7))
   (segment (start 210.82 104.14) (end 213.36 104.14) (width 0.75) (layer B.Cu) (net 7))
   (segment (start 213.36 104.14) (end 214.63 102.87) (width 0.75) (layer B.Cu) (net 7))
@@
   (segment (start 220.98 118.11) (end 220.98 119.38) (width 0.75) (layer B.Cu) (net 7))
   (segment (start 219.71 116.84) (end 220.98 118.11) (width 0.75) (layer B.Cu) (net 7))
-  (segment (start 246.38 161.29) (end 246.38 163.83) (width 0.75) (layer B.Cu) (net 7))
   (segment (start 233.68 104.14) (end 236.22 104.14) (width 0.75) (layer B.Cu) (net 7))
   (segment (start 236.22 116.84) (end 233.68 116.84) (width 0.75) (layer B.Cu) (net 7))
@@
   (segment (start 237.49 189.23) (end 236.22 187.96) (width 1.5) (layer B.Cu) (net 38))
   (segment (start 236.22 187.96) (end 233.68 185.42) (width 1.5) (layer B.Cu) (net 38))
+  (zone (net 1) (net_name /ALIM/GND) (layer B.Cu) (hatch edge 0.508)
+    (connect_pads (clearance 0.508))
+    (min_thickness 0.254)
+    (fill (arc_segments 16) (thermal_gap 0.508) (thermal_bridge_width 0.508))
+    (polygon
+      (pts
+        (xy 281.94 201.93) (xy 160.02 201.93) (xy 160.02 73.66) (xy 281.94 73.66)
+      )
+    )
+  )
+  (zone (net 1) (net_name /ALIM/GND) (layer F.Cu) (hatch edge 0.508)
+    (connect_pads (clearance 0.508))
+    (min_thickness 0.254)
+    (fill (arc_segments 16) (thermal_gap 0.508) (thermal_bridge_width 0.508))
+    (polygon
+      (pts
+        (xy 281.94 201.93) (xy 160.02 201.93) (xy 160.02 73.66) (xy 281.94 73.66)
+      )
+    )
+  )
 )

Commit message: Shield V2 (PCB begining)
Parts:
- removed C10, C11, C12, C5, C6, C7, C8, C9: C, C2
- moved C2 63.8 mm to (188.0, 111.8)
- moved C1 56.0 mm to (256.5, 111.8)
- moved GP2_LB1 29.2 mm to (210.8, 141.0)
- moved GP2_LF1 29.2 mm to (210.8, 129.5)
- moved GP2_RB1 29.2 mm to (210.8, 137.2)
- moved GP2_RF1 29.2 mm to (210.8, 133.3)
- moved SERVO_LB0 22.9 mm to (185.4, 157.5), turned to 0 degrees
- moved SERVO_LB2 22.9 mm to (185.4, 167.6), turned to 0 degrees
- moved SERVO_LB1 22.9 mm to (185.4, 162.6), turned to 0 degrees
- moved GPIO1 21.7 mm to (205.7, 149.9)
- moved SERVO_LF0 19.4 mm to (185.4, 100.3), turned to 0 degrees
- moved SERVO_LF1 19.4 mm to (185.4, 95.2), turned to 0 degrees
- moved SERVO_LF2 19.4 mm to (185.4, 90.2), turned to 0 degrees
- moved SERVO_RB0 18.9 mm to (260.4, 157.5), turned to 180 degrees
- moved SERVO_RB2 18.9 mm to (260.4, 167.6), turned to 180 degrees
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Connections:
- net N-0000078 renamed /ALIM/EN
- ALIM_BOARD1 pad 2: N-0000079 (its old number) -> /ALIM/BAT
- GP2_LB1 pad 1: /ARDUINO/GP2_LB -> /ALIM/GND
- GP2_LB1 pad 3: /ALIM/GND -> /ARDUINO/GP2_LB
- GP2_LF1 pad 1: /ARDUINO/GP2_LF -> /ALIM/GND
- GP2_LF1 pad 3: /ALIM/GND -> /ARDUINO/GP2_LF
- GP2_RB1 pad 1: /ARDUINO/GP2_RB -> /ALIM/GND
- GP2_RB1 pad 3: /ALIM/GND -> /ARDUINO/GP2_RB
- GP2_RF1 pad 1: /ARDUINO/GP2_RF -> /ALIM/GND
- GP2_RF1 pad 3: /ALIM/GND -> /ARDUINO/GP2_RF
- SECURITY_SWITCH1 pad 2: N-0000079 (its old number) -> /ALIM/BAT
- SERVO_LB0 pad 1: /LEG_RB/PWM0 -> /ALIM/GND
- SERVO_LB0 pad 3: /ALIM/GND -> /LEG_LB/PWM0
- SERVO_LB1 pad 1: /LEG_RB/PWM2 -> /ALIM/GND
- SERVO_LB1 pad 3: /ALIM/GND -> /LEG_LB/PWM1
- SERVO_LB2 pad 1: /LEG_RB/PWM1 -> /ALIM/GND
- SERVO_LB2 pad 3: /ALIM/GND -> /LEG_LB/PWM2
- SERVO_LF0 pad 1: /LEG_LF/PWM0 -> /ALIM/GND
- SERVO_LF0 pad 3: /ALIM/GND -> /LEG_LF/PWM0
- SERVO_LF1 pad 1: /LEG_LF/PWM2 -> /ALIM/GND
- SERVO_LF1 pad 3: /ALIM/GND -> /LEG_LF/PWM1
- SERVO_LF2 pad 1: /LEG_LF/PWM1 -> /ALIM/GND
- SERVO_LF2 pad 3: /ALIM/GND -> /LEG_LF/PWM2
- SERVO_RB0 pad 1: /LEG_LB/PWM0 -> /ALIM/GND
- SERVO_RB0 pad 3: /ALIM/GND -> /LEG_RB/PWM0
- SERVO_RB1 pad 1: /LEG_LB/PWM2 -> /ALIM/GND
- SERVO_RB1 pad 3: /ALIM/GND -> /LEG_RB/PWM1
- SERVO_RB2 pad 1: /LEG_LB/PWM1 -> /ALIM/GND
- SERVO_RB2 pad 3: /ALIM/GND -> /LEG_RB/PWM2
- SERVO_RF0 pad 1: /LEG_RF/PWM0 -> /ALIM/GND
- SERVO_RF0 pad 3: /ALIM/GND -> /LEG_RF/PWM0
- SERVO_RF1 pad 1: /LEG_RF/PWM1 -> /ALIM/GND
- SERVO_RF1 pad 3: /ALIM/GND -> /LEG_RF/PWM1
- SERVO_RF2 pad 1: /LEG_RF/PWM2 -> /ALIM/GND
- SERVO_RF2 pad 3: /ALIM/GND -> /LEG_RF/PWM2
- SHIELD1 pad 2: /LEG_RF/PWM1 -> /LEG_RB/PWM2
- SHIELD1 pad 3: /LEG_RF/PWM2 -> /LEG_RB/PWM1
- SHIELD1 pad 5: /LEG_RF/PWM0 -> /LEG_RB/PWM0
- SHIELD1 pad 6: /LEG_RB/PWM0 -> /LEG_RF/PWM0
- SHIELD1 pad 7: /LEG_RB/PWM1 -> /LEG_RF/PWM1
- SHIELD1 pad 8: /LEG_RB/PWM2 -> /LEG_RF/PWM2
- SPI1 pad 10: /ARDUINO/MISO -> /ARDUINO/SS
- SPI1 pad 4: /ARDUINO/SS -> /ARDUINO/MOSI
- SPI1 pad 6: /ARDUINO/SCK -> /ARDUINO/MISO
- SPI1 pad 8: /ARDUINO/MOSI -> /ARDUINO/SCK
- UART1 pad 1: /ARDUINO/RX -> /ALIM/GND
- UART1 pad 3: /ALIM/GND -> /ARDUINO/RX
Routing:
- net /ALIM/POW_5V: track 526.7 -> 0.00 mm
- net /ARDUINO/LOG_5V: track 190.7 -> 0.00 mm
- net /LEG_RB/PWM1: track 156.0 -> 0.00 mm, vias 1 -> 0
- net /LEG_RB/PWM2: track 152.2 -> 0.00 mm, vias 3 -> 0
- net /ARDUINO/SCL: track 123.9 -> 0.00 mm
- net /LEG_RB/PWM0: track 117.9 -> 0.00 mm
- net /ARDUINO/SDA: track 116.0 -> 0.00 mm, vias 2 -> 0
- net /LEG_LF/PWM2: track 106.3 -> 0.00 mm, vias 1 -> 0
- net /LEG_LF/PWM1: track 99.4 -> 0.00 mm
- net /LEG_LF/PWM0: track 92.5 -> 0.00 mm, vias 1 -> 0
- net /LEG_LB/PWM1: track 81.2 -> 0.00 mm
- net /LEG_RF/PWM1: track 77.7 -> 0.00 mm
- net /LEG_LB/PWM2: track 77.2 -> 0.00 mm
- net /LEG_RF/PWM2: track 73.6 -> 0.00 mm
- net /LEG_LB/PWM0: track 72.9 -> 0.00 mm, vias 1 -> 0
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- removed copper zone on B.Cu, net /ALIM/GND
- removed copper zone on F.Cu, net /ALIM/GND

Commit message: Before routing.
Parts:
- moved SERVO_RB0 1.27 mm to (259.1, 157.5)
- moved SERVO_RB1 1.27 mm to (259.1, 162.6)
- moved SERVO_RB2 1.27 mm to (259.1, 167.6)
- moved C3 1.27 mm to (256.5, 176.5)
Changed lines of the file:
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@@
     (user_trace_width 1.25)
     (user_trace_width 1.5)
+    (user_trace_width 1.75)
     (trace_clearance 0.254)
     (zone_clearance 0.508)
@@
   )
   (module C2 (layer F.Cu)
-    (at 257.81 176.53 180)
+    (at 256.54 176.53 180)
     (descr "Condensateur = 2 pas")
     (tags C)
@@
   )
   (module PIN_ARRAY_3X1 (layer F.Cu)
-    (at 260.35 162.56 180)
+    (at 259.08 162.56 180)
     (descr "Connecteur 3 pins")
     (tags "CONN DEV")
@@
   )
   (module PIN_ARRAY_3X1 (layer F.Cu)
-    (at 260.35 167.64 180)
+    (at 259.08 167.64 180)
     (descr "Connecteur 3 pins")
     (tags "CONN DEV")
@@
   )
   (module PIN_ARRAY_3X1 (layer F.Cu)
-    (at 260.35 157.48 180)
-    (descr "Connecteur 3 pins")
-    (tags "CONN DEV")
+    (at 259.08 157.48 180)
+    (descr "Connecteur 3 pins")
+    (tags "CONN DEV")

Commit message: PCB almost finished !
Parts:
- moved I2C0 3.81 mm to (222.2, 105.4)
- moved I2C1 3.81 mm to (222.2, 109.2)
Routing:
- net /ALIM/POW_5V: track 0.00 -> 262.0 mm
- net /ARDUINO/LOG_5V: track 0.00 -> 102.6 mm
- net /LEG_LF/PWM2: track 0.00 -> 68.3 mm
- net /LEG_LF/PWM0: track 0.00 -> 68.3 mm
- net /ARDUINO/SCL: track 0.00 -> 67.8 mm
- net /LEG_LF/PWM1: track 0.00 -> 67.3 mm
- net /ARDUINO/SDA: track 0.00 -> 63.5 mm
- net /LEG_RB/PWM2: track 0.00 -> 46.9 mm
- net /LEG_RB/PWM0: track 0.00 -> 45.1 mm
- net /LEG_RB/PWM1: track 0.00 -> 44.3 mm
- net /LEG_LB/PWM2: track 0.00 -> 40.6 mm
- net /LEG_LB/PWM0: track 0.00 -> 37.4 mm
- net /LEG_LB/PWM1: track 0.00 -> 34.5 mm
- net /ALIM/BAT: track 0.00 -> 27.3 mm
- net /LEG_RF/PWM2: track 0.00 -> 23.9 mm
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
Commit message: PCB FINISHED ! + Correction of schematics.
Connections:
- SHIELD1 pad GND1: /ALIM/GND -> (no net)
Routing:
- added copper zone on B.Cu, net /ALIM/GND
- added copper zone on F.Cu, net /ALIM/GND
Changed lines of the file:
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@@
 (kicad_pcb (version 3) (host pcbnew "(2013-june-11)-stable")
   (general
-    (links 117)
-    (no_connects 40)
+    (links 112)
+    (no_connects 0)
     (area 160.02 64.786934 281.940001 201.930001)
     (thickness 1.6)
@@
   (net 36 /LEG_RF/PWM1)
   (net 37 /LEG_RF/PWM2)
-  (net 38 N-0000079)
+  (net 38 N-0000080)
   (net_class Default "Ceci est la Netclass par défaut"
     (clearance 0.254)
@@
     (add_net /LEG_RF/PWM1)
     (add_net /LEG_RF/PWM2)
-    (add_net N-0000079)
+    (add_net N-0000080)
   )
   (module ARDUINO_MEGA_SHIELD (layer F.Cu)
@@
     (pad GND1 thru_hole oval (at 40.64 -2.54) (size 2.54 1.524) (drill 0.8128)
       (layers *.Cu *.Mask F.SilkS)
-      (net 3 /ALIM/GND)
     )
     (pad 3V3 thru_hole oval (at 35.56 -2.54) (size 2.54 1.524) (drill 0.8128)
@@
     (pad GND1 thru_hole circle (at 96.52 -2.54) (size 3.937 3.937) (drill 3.175)
       (layers *.Cu *.Mask F.SilkS)
-      (net 3 /ALIM/GND)
     )
     (pad GND1 thru_hole circle (at 90.17 -50.8) (size 3.937 3.937) (drill 3.175)
       (layers *.Cu *.Mask F.SilkS)
-      (net 3 /ALIM/GND)
     )
     (pad GND1 thru_hole circle (at 15.24 -50.8) (size 3.937 3.937) (drill 3.175)
       (layers *.Cu *.Mask F.SilkS)
-      (net 3 /ALIM/GND)
     )
     (pad GND1 thru_hole circle (at 13.97 -2.54) (size 3.937 3.937) (drill 3.175)
       (layers *.Cu *.Mask F.SilkS)
-      (net 3 /ALIM/GND)
     )
     (pad 22 thru_hole circle (at 93.98 -48.26 270) (size 1.524 1.524) (drill 0.8128)
@@
     (pad 1 thru_hole circle (at 3.81 -2.54 180) (size 1.397 1.397) (drill 0.8128)
       (layers *.Cu *.Mask F.SilkS)
-      (net 38 N-0000079)
+      (net 38 N-0000080)
     )
     (pad 2 thru_hole circle (at 3.81 2.54 180) (size 1.397 1.397) (drill 0.8128)
@@
     (pad 1 thru_hole circle (at -3.81 -2.54 180) (size 1.397 1.397) (drill 0.8128)
       (layers *.Cu *.Mask F.SilkS)
-      (net 38 N-0000079)
+      (net 38 N-0000080)
     )
     (pad 2 thru_hole circle (at -3.81 2.54 180) (size 1.397 1.397) (drill 0.8128)
@@
     (pad 2 thru_hole circle (at 0 0) (size 1.524 1.524) (drill 1.016)
       (layers *.Cu *.Mask F.SilkS)
-      (net 38 N-0000079)
+      (net 38 N-0000080)
     )
     (pad 3 thru_hole circle (at 2.54 0) (size 1.524 1.524) (drill 1.016)
@@
   (segment (start 231.14 176.53) (end 223.52 184.15) (width 1.75) (layer B.Cu) (net 1))
   (segment (start 223.52 184.15) (end 214.63 184.15) (width 1.75) (layer B.Cu) (net 1))
-  (segment (start 214.63 186.69) (end 214.63 191.77) (width 1) (layer B.Cu) (net 2) (status C00000))
+  (segment (start 214.63 186.69) (end 214.63 191.77) (width 1) (layer B.Cu) (net 2))
   (segment (start 185.42 176.53) (end 185.42 167.64) (width 1.75) (layer B.Cu) (net 4))
   (segment (start 214.63 176.53) (end 200.66 176.53) (width 1.75) (layer B.Cu) (net 4))
@@
   (segment (start 231.14 83.82) (end 213.36 83.82) (width 1) (layer B.Cu) (net 31))
   (segment (start 243.586 96.266) (end 231.14 83.82) (width 1) (layer B.Cu) (net 31))
-  (segment (start 246.38 118.11) (end 248.92 118.11) (width 1) (layer B.Cu) (net 32) (status 400000))
-  (segment (start 255.27 156.21) (end 256.54 157.48) (width 1) (layer B.Cu) (net 32) (status 800000))
+  (segment (start 246.38 118.11) (end 248.92 118.11) (width 1) (layer B.Cu) (net 32))
+  (segment (start 255.27 156.21) (end 256.54 157.48) (width 1) (layer B.Cu) (net 32))
   (segment (start 255.27 124.46) (end 255.27 156.21) (width 1) (layer B.Cu) (net 32))
   (segment (start 248.92 118.11) (end 255.27 124.46) (width 1) (layer B.Cu) (net 32))
-  (segment (start 246.38 123.19) (end 247.65 123.19) (width 1) (layer B.Cu) (net 33) (status C00000))
-  (segment (start 252.73 158.75) (end 256.54 162.56) (width 1) (layer B.Cu) (net 33) (status 800000))
+  (segment (start 246.38 123.19) (end 247.65 123.19) (width 1) (layer B.Cu) (net 33))
+  (segment (start 252.73 158.75) (end 256.54 162.56) (width 1) (layer B.Cu) (net 33))
   (segment (start 252.73 128.27) (end 252.73 158.75) (width 1) (layer B.Cu) (net 33))
-  (segment (start 247.65 123.19) (end 252.73 128.27) (width 1) (layer B.Cu) (net 33) (status 400000))
-  (segment (start 246.38 125.73) (end 247.65 125.73) (width 1) (layer B.Cu) (net 34) (status C00000))
-  (segment (start 250.19 161.29) (end 256.54 167.64) (width 1) (layer B.Cu) (net 34) (status 800000))
+  (segment (start 247.65 123.19) (end 252.73 128.27) (width 1) (layer B.Cu) (net 33))
+  (segment (start 246.38 125.73) (end 247.65 125.73) (width 1) (layer B.Cu) (net 34))
+  (segment (start 250.19 161.29) (end 256.54 167.64) (width 1) (layer B.Cu) (net 34))
   (segment (start 250.19 128.27) (end 250.19 161.29) (width 1) (layer B.Cu) (net 34))
-  (segment (start 247.65 125.73) (end 250.19 128.27) (width 1) (layer B.Cu) (net 34) (status 400000))
-  (segment (start 246.38 115.57) (end 247.65 115.57) (width 1) (layer B.Cu) (net 35) (status C00000))
-  (segment (start 256.54 105.41) (end 256.54 100.33) (width 1) (layer B.Cu) (net 35) (status 800000))
+  (segment (start 247.65 125.73) (end 250.19 128.27) (width 1) (layer B.Cu) (net 34))
+  (segment (start 246.38 115.57) (end 247.65 115.57) (width 1) (layer B.Cu) (net 35))
+  (segment (start 256.54 105.41) (end 256.54 100.33) (width 1) (layer B.Cu) (net 35))
   (segment (start 251.46 110.49) (end 256.54 105.41) (width 1) (layer B.Cu) (net 35))
   (segment (start 251.46 111.76) (end 251.46 110.49) (width 1) (layer B.Cu) (net 35))
-  (segment (start 247.65 115.57) (end 251.46 111.76) (width 1) (layer B.Cu) (net 35) (status 400000))
-  (segment (start 246.38 113.03) (end 247.65 113.03) (width 1) (layer B.Cu) (net 36) (status C00000))
-  (segment (start 254 97.79) (end 256.54 95.25) (width 1) (layer B.Cu) (net 36) (status 800000))
+  (segment (start 247.65 115.57) (end 251.46 111.76) (width 1) (layer B.Cu) (net 35))
+  (segment (start 246.38 113.03) (end 247.65 113.03) (width 1) (layer B.Cu) (net 36))
+  (segment (start 254 97.79) (end 256.54 95.25) (width 1) (layer B.Cu) (net 36))
   (segment (start 254 105.41) (end 254 97.79) (width 1) (layer B.Cu) (net 36))
   (segment (start 250.19 109.22) (end 254 105.41) (width 1) (layer B.Cu) (net 36))
   (segment (start 250.19 110.49) (end 250.19 109.22) (width 1) (layer B.Cu) (net 36))
-  (segment (start 247.65 113.03) (end 250.19 110.49) (width 1) (layer B.Cu) (net 36) (status 400000))
-  (segment (start 246.38 108.966) (end 247.904 108.966) (width 1) (layer B.Cu) (net 37) (status 400000))
-  (segment (start 251.46 95.25) (end 256.54 90.17) (width 1) (layer B.Cu) (net 37) (status 800000))
+  (segment (start 247.65 113.03) (end 250.19 110.49) (width 1) (layer B.Cu) (net 36))
+  (segment (start 246.38 108.966) (end 247.904 108.966) (width 1) (layer B.Cu) (net 37))
+  (segment (start 251.46 95.25) (end 256.54 90.17) (width 1) (layer B.Cu) (net 37))
   (segment (start 251.46 105.41) (end 251.46 95.25) (width 1) (layer B.Cu) (net 37))
   (segment (start 247.904 108.966) (end 251.46 105.41) (width 1) (layer B.Cu) (net 37))
@@
   (segment (start 231.14 189.23) (end 231.14 186.69) (width 1.75) (layer B.Cu) (net 38))
   (segment (start 231.14 186.69) (end 231.14 181.61) (width 1.75) (layer B.Cu) (net 38))
+  (zone (net 3) (net_name /ALIM/GND) (layer B.Cu) (hatch edge 0.508)
+    (connect_pads thru_hole_only (clearance 0.508))
+    (min_thickness 0.254)
+    (fill (arc_segments 16) (thermal_gap 0.508) (thermal_bridge_width 0.508) (smoothing chamfer))
+    (polygon
+      (pts
+        (xy 222.25 82.55) (xy 180.34 82.55) (xy 180.34 180.34) (xy 194.31 194.31) (xy 247.65 194.31)
+        (xy 250.19 194.31) (xy 264.16 180.34) (xy 264.16 82.55) (xy 222.25 82.55)
+      )
+    )
+  )
+  (zone (net 3) (net_name /ALIM/GND) (layer F.Cu) (hatch edge 0.508)
+    (connect_pads thru_hole_only (clearance 0.508))
+    (min_thickness 0.254)
+    (fill (arc_segments 16) (thermal_gap 0.508) (thermal_bridge_width 0.508) (smoothing chamfer))
+    (polygon
+      (pts
+        (xy 264.16 180.34) (xy 250.19 194.31) (xy 194.31 194.31) (xy 180.34 180.34) (xy 180.34 82.55)
+        (xy 264.16 82.55)
+      )
+    )
+  )
 )

Commit message: PCB v3 !
Parts:
- moved POW_BATTERY1 18.3 mm to (246.4, 181.6), turned to 90 degrees
- moved R_SCL1 17.3 mm to (233.7, 109.2)
- moved R_SDA1 14.9 mm to (231.1, 109.2)
- moved ENABLE_ALIM1 13.7 mm to (226.1, 184.2)
- moved SERVO_LB1 8.89 mm to (185.4, 153.7)
- moved SERVO_RB1 8.89 mm to (259.1, 153.7)
- moved SERVO_LB0 8.89 mm to (185.4, 148.6)
- moved SERVO_LB2 8.89 mm to (185.4, 158.8)
- moved SERVO_RB0 8.89 mm to (259.1, 148.6)
- moved SERVO_RB2 8.89 mm to (259.1, 158.8)
- moved ALIM_BOARD1 6.84 mm to (221.0, 179.1)
- moved C4 6.84 mm to (185.4, 170.2), turned to 270 degrees
- moved C3 6.84 mm to (259.1, 170.2), turned to 270 degrees
- moved C1 3.81 mm to (256.5, 115.6)
- moved C2 3.81 mm to (188.0, 115.6)
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Routing:
- net /ALIM/POW_5V: track 262.0 -> 236.0 mm
- net /ARDUINO/LOG_5V: track 102.6 -> 117.0 mm
- net /ARDUINO/SCL: track 67.8 -> 79.8 mm
- net /LEG_RB/PWM0: track 45.1 -> 35.4 mm
- net /LEG_LB/PWM1: track 34.5 -> 43.4 mm
- net /LEG_LB/PWM0: track 37.4 -> 46.3 mm
- net /LEG_RB/PWM2: track 46.9 -> 38.0 mm
- net /ALIM/BAT: track 27.3 -> 18.8 mm
- net /LEG_RB/PWM1: track 44.3 -> 36.2 mm
- net /LEG_LF/PWM1: track 67.3 -> 59.9 mm
- net /LEG_LF/PWM0: track 68.3 -> 60.9 mm
- net /LEG_LF/PWM2: track 68.3 -> 60.9 mm
- net N-0000080: track 23.5 -> 16.3 mm
- net /LEG_LB/PWM2: track 40.6 -> 47.3 mm
- net /ARDUINO/SDA: track 63.5 -> 65.8 mm
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