File: elec/adm_shield/adm_shield.kicad_pcb (KiCad board)
At the start: 2 copper layers, 35 parts

Commit message: V3.1 ?
Parts:
- added C5: C, C2, F.Cu at (243.8, 176.5)
- moved POW_BATTERY1 6.35 mm to (250.2, 176.5)
- moved ENABLE_ALIM1 5.08 mm to (226.1, 179.1)
- moved SECURITY_SWITCH1 5.08 mm to (234.9, 176.5)
- moved ALIM_BOARD1 5.08 mm to (221.0, 174.0)
Connections:
- ALIM_BOARD1 pad 2: /ALIM/BAT -> N-0000080
- POW_BATTERY1 pad 2: N-0000080 -> /ALIM/BAT
- SECURITY_SWITCH1 pad 1: N-0000080 -> /ALIM/BAT
- SECURITY_SWITCH1 pad 2: /ALIM/BAT -> N-0000080
Routing:
- net N-0000080: track 16.3 -> 18.8 mm
- net /ALIM/BAT: track 18.8 -> 20.1 mm
Changed lines of the file:
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@@
 (kicad_pcb (version 3) (host pcbnew "(2013-07-07 BZR 4022)-stable")
   (general
-    (links 112)
+    (links 114)
     (no_connects 0)
-    (area 180.2638 64.786934 264.2362 194.310001)
+    (area 0 0 0 0)
     (thickness 1.6)
     (drawings 0)
     (tracks 213)
     (zones 0)
-    (modules 35)
+    (modules 36)
     (nets 39)
   )
   (page A3)
   (layers
-    (15 F.Cu signal hide)
+    (15 F.Cu signal)
     (0 B.Cu signal)
     (16 Dessous.Adhes user)
@@
   )
   (setup
-    (last_trace_width 1)
+    (last_trace_width 1.75)
     (user_trace_width 0.5)
     (user_trace_width 0.75)
@@
     (trace_clearance 0.254)
     (zone_clearance 0.508)
-    (zone_45_only no)
+    (zone_45_only yes)
     (trace_min 0.254)
     (segment_width 0.2)
@@
     (mod_text_size 1.5 1.5)
     (mod_text_width 0.15)
-    (pad_size 1.524 1.524)
+    (pad_size 1.724 1.724)
     (pad_drill 0.762)
     (pad_to_mask_clearance 0.2)
@@
   )
   (module SW_PUSH_SMALL (layer F.Cu)
-    (at 234.95 181.61 180)
+    (at 234.95 176.53 180)
     (fp_text reference SECURITY_SWITCH1 (at 0 -0.762 180) (layer Dessus.SilkS)
       (effects (font (size 1.016 1.016) (thickness 0.2032)))
@@
     (pad 1 thru_hole circle (at 3.81 -2.54 180) (size 1.397 1.397) (drill 0.8128)
       (layers *.Cu *.Mask Dessus.SilkS)
+      (net 1 /ALIM/BAT)
+    )
+    (pad 2 thru_hole circle (at 3.81 2.54 180) (size 1.397 1.397) (drill 0.8128)
+      (layers *.Cu *.Mask Dessus.SilkS)
       (net 38 N-0000080)
     )
-    (pad 2 thru_hole circle (at 3.81 2.54 180) (size 1.397 1.397) (drill 0.8128)
+    (pad 1 thru_hole circle (at -3.81 -2.54 180) (size 1.397 1.397) (drill 0.8128)
       (layers *.Cu *.Mask Dessus.SilkS)
       (net 1 /ALIM/BAT)
     )
-    (pad 1 thru_hole circle (at -3.81 -2.54 180) (size 1.397 1.397) (drill 0.8128)
+    (pad 2 thru_hole circle (at -3.81 2.54 180) (size 1.397 1.397) (drill 0.8128)
       (layers *.Cu *.Mask Dessus.SilkS)
       (net 38 N-0000080)
-    )
-    (pad 2 thru_hole circle (at -3.81 2.54 180) (size 1.397 1.397) (drill 0.8128)
-      (layers *.Cu *.Mask Dessus.SilkS)
-      (net 1 /ALIM/BAT)
     )
   )
@@
   )
   (module PIN_ARRAY_5x1 (layer F.Cu)
-    (at 220.98 179.07 90)
+    (at 220.98 173.99 90)
     (descr "Double rangee de contacts 2 x 5 pins")
     (tags CONN)
@@
     (pad 2 thru_hole circle (at -2.54 0 90) (size 1.524 1.524) (drill 1.016)
       (layers *.Cu *.Mask Dessus.SilkS)
-      (net 1 /ALIM/BAT)
+      (net 38 N-0000080)
     )
     (pad 3 thru_hole circle (at 0 0 90) (size 1.524 1.524) (drill 1.016)
@@
   )
   (module PIN_ARRAY_3X1 (layer F.Cu)
-    (at 246.38 181.61 90)
+    (at 250.19 176.53 90)
     (descr "Connecteur 3 pins")
     (tags "CONN DEV")
@@
     (pad 2 thru_hole circle (at 0 0 90) (size 1.524 1.524) (drill 1.016)
       (layers *.Cu *.Mask Dessus.SilkS)
-      (net 38 N-0000080)
+      (net 1 /ALIM/BAT)
     )
     (pad 3 thru_hole circle (at 2.54 0 90) (size 1.524 1.524) (drill 1.016)
@@
   )
   (module PIN_ARRAY_1 (layer F.Cu)
-    (at 226.06 184.15)
+    (at 226.06 179.07)
     (descr "1 pin")
     (tags "CONN DEV")
@@
     )
   )
-  (segment (start 231.14 179.07) (end 228.6 179.07) (width 1.75) (layer B.Cu) (net 1))
-  (segment (start 226.06 181.61) (end 220.98 181.61) (width 1.75) (layer B.Cu) (net 1))
-  (segment (start 228.6 179.07) (end 226.06 181.61) (width 1.75) (layer B.Cu) (net 1))
+  (module C2 (layer F.Cu)
+    (at 243.84 176.53 90)
+    (descr "Condensateur = 2 pas")
+    (tags C)
+    (fp_text reference C5 (at 0 0 90) (layer Dessus.SilkS)
+      (effects (font (size 1.016 1.016) (thickness 0.2032)))
+    )
+    (fp_text value C (at 0 0 90) (layer Dessus.SilkS) hide
+      (effects (font (size 1.016 1.016) (thickness 0.2032)))
+    )
+    (fp_line (start -3.556 -1.016) (end 3.556 -1.016) (layer Dessus.SilkS) (width 0.3048))
+    (fp_line (start 3.556 -1.016) (end 3.556 1.016) (layer Dessus.SilkS) (width 0.3048))
+    (fp_line (start 3.556 1.016) (end -3.556 1.016) (layer Dessus.SilkS) (width 0.3048))
+    (fp_line (start -3.556 1.016) (end -3.556 -1.016) (layer Dessus.SilkS) (width 0.3048))
+    (fp_line (start -3.556 -0.508) (end -3.048 -1.016) (layer Dessus.SilkS) (width 0.3048))
+    (pad 1 thru_hole circle (at -2.54 0 90) (size 1.397 1.397) (drill 0.8128)
+      (layers *.Cu *.Mask Dessus.SilkS)
+      (net 1 /ALIM/BAT)
+    )
+    (pad 2 thru_hole circle (at 2.54 0 90) (size 1.397 1.397) (drill 0.8128)
+      (layers *.Cu *.Mask Dessus.SilkS)
+      (net 3 /ALIM/GND)
+    )
+    (model discret/capa_2pas_5x5mm.wrl
+      (at (xyz 0 0 0))
+      (scale (xyz 1 1 1))
+      (rotate (xyz 0 0 0))
+    )
+  )
+  (segment (start 250.19 176.53) (end 246.38 176.53) (width 1.75) (layer B.Cu) (net 1))
+  (segment (start 246.38 176.53) (end 243.84 179.07) (width 1.75) (layer B.Cu) (net 1))
+  (segment (start 243.84 179.07) (end 238.76 179.07) (width 1.75) (layer B.Cu) (net 1) (status 10))
   (segment (start 238.76 179.07) (end 231.14 179.07) (width 1.75) (layer B.Cu) (net 1) (status 30))
-  (segment (start 220.98 184.15) (end 226.06 184.15) (width 1) (layer B.Cu) (net 2))
-  (segment (start 259.08 167.64) (end 252.73 173.99) (width 1.75) (layer B.Cu) (net 4))
-  (segment (start 252.73 173.99) (end 220.98 173.99) (width 1.75) (layer B.Cu) (net 4))
+  (segment (start 220.98 179.07) (end 226.06 179.07) (width 1) (layer B.Cu) (net 2))
+  (segment (start 220.98 168.91) (end 257.81 168.91) (width 1.75) (layer B.Cu) (net 4))
+  (segment (start 257.81 168.91) (end 259.08 167.64) (width 1.75) (layer B.Cu) (net 4))
   (segment (start 185.42 167.64) (end 194.31 176.53) (width 1.75) (layer B.Cu) (net 4))
-  (segment (start 194.31 176.53) (end 203.2 176.53) (width 1.75) (layer B.Cu) (net 4))
-  (segment (start 215.9 173.99) (end 220.98 173.99) (width 1.75) (layer B.Cu) (net 4))
-  (segment (start 213.36 176.53) (end 203.2 176.53) (width 1.75) (layer B.Cu) (net 4))
-  (segment (start 215.9 173.99) (end 213.36 176.53) (width 1.75) (layer B.Cu) (net 4))
+  (segment (start 218.44 168.91) (end 210.82 176.53) (width 1.75) (layer B.Cu) (net 4))
+  (segment (start 210.82 176.53) (end 201.93 176.53) (width 1.75) (layer B.Cu) (net 4))
+  (segment (start 218.44 168.91) (end 220.98 168.91) (width 1.75) (layer B.Cu) (net 4))
+  (segment (start 194.31 176.53) (end 201.93 176.53) (width 1.75) (layer B.Cu) (net 4))
   (segment (start 185.42 167.64) (end 185.42 158.75) (width 1.75) (layer B.Cu) (net 4) (status 10))
   (segment (start 259.08 167.64) (end 259.08 158.75) (width 1.75) (layer B.Cu) (net 4) (status 10))
@@
   (segment (start 251.46 105.41) (end 251.46 95.25) (width 1) (layer B.Cu) (net 37))
   (segment (start 247.904 108.966) (end 251.46 105.41) (width 1) (layer B.Cu) (net 37))
-  (segment (start 238.76 184.15) (end 241.3 184.15) (width 1.75) (layer B.Cu) (net 38))
-  (segment (start 243.84 181.61) (end 246.38 181.61) (width 1.75) (layer B.Cu) (net 38))
-  (segment (start 241.3 184.15) (end 243.84 181.61) (width 1.75) (layer B.Cu) (net 38))
-  (segment (start 238.76 184.15) (end 231.14 184.15) (width 1.75) (layer B.Cu) (net 38) (status 30))
+  (segment (start 231.14 173.99) (end 226.06 173.99) (width 1.75) (layer B.Cu) (net 38))
+  (segment (start 223.52 176.53) (end 220.98 176.53) (width 1.75) (layer B.Cu) (net 38))
+  (segment (start 226.06 173.99) (end 223.52 176.53) (width 1.75) (layer B.Cu) (net 38))
+  (segment (start 238.76 173.99) (end 231.14 173.99) (width 1.75) (layer B.Cu) (net 38) (status 30))
   (zone (net 3) (net_name /ALIM/GND) (layer B.Cu) (hatch edge 0.508)
     (connect_pads (clearance 0.508))
@@
     (polygon
       (pts
-        (xy 264.16 187.96) (xy 180.34 187.96) (xy 180.34 87.63) (xy 264.16 87.63)
+        (xy 264.16 182.88) (xy 180.34 182.88) (xy 180.34 87.63) (xy 264.16 87.63)
       )
     )
@@
     (polygon
       (pts
-        (xy 264.16 187.96) (xy 180.34 187.96) (xy 180.34 87.63) (xy 264.16 87.63)
+        (xy 264.16 182.88) (xy 180.34 182.88) (xy 180.34 87.63) (xy 264.16 87.63)
       )
     )
+  )
+  (zone (net 0) (net_name "") (layer B.Cu) (hatch edge 0.508)
+    (connect_pads (clearance 0.508))
+    (min_thickness 0.254)
+    (keepout (tracks not_allowed) (vias not_allowed) (copperpour allowed))
+    (fill (arc_segments 16) (thermal_gap 0.508) (thermal_bridge_width 0.508))
+    (polygon
+      (pts
+        (xy 228.6 144.78) (xy 218.44 144.78) (xy 218.44 128.27) (xy 228.6 128.27)
+      )
+    )
+  )
+  (zone (net 0) (net_name "") (layer F.Cu) (hatch edge 0.508)
+    (connect_pads (clearance 0.508))
+    (min_thickness 0.254)
+    (keepout (tracks not_allowed) (vias not_allowed) (copperpour allowed))
+    (fill (arc_segments 16) (thermal_gap 0.508) (thermal_bridge_width 0.508))
+    (polygon
+      (pts
+        (xy 228.6 144.78) (xy 218.44 144.78) (xy 218.44 128.27) (xy 228.6 128.27)
+      )
+    )
