File: elec/adm_shield/adm_shield.kicad_pcb (KiCad board)
At the start: 2 copper layers, 35 parts

Commit message: New wlaking algo. PCB v4
Routing:
- net /ARDUINO/GP2_LB: track 16.3 -> 14.8 mm
- net /ARDUINO/LOG_5V: track 102.6 -> 103.4 mm
- net /ARDUINO/GP2_RB: track 16.1 -> 15.3 mm
- net (no net): vias 0 -> 21
- added copper zone on B.Cu, net /ALIM/POW_5V
Other:
- net class Default: clearance 0.254 -> 0.25; via_dia 0.889 -> 0.89
- rule trace_clearance: 0.254 -> 0.25
