File: elec/adm_shield/adm_shield.kicad_pcb (KiCad board)
At the start: 2 copper layers, 35 parts

Commit message: PCB v4.1
Parts:
- added C5: C, C2, F.Cu at (243.8, 176.5)
- moved POW_BATTERY1 24.4 mm to (250.2, 176.5), turned to 90 degrees
- moved R_SCL1 17.3 mm to (233.7, 109.2)
- moved ENABLE_ALIM1 17.1 mm to (226.1, 179.1)
- moved R_SDA1 14.9 mm to (231.1, 109.2)
- moved ALIM_BOARD1 9.92 mm to (221.0, 174.0)
- moved SERVO_LB1 8.89 mm to (185.4, 153.7)
- moved SERVO_RB1 8.89 mm to (259.1, 153.7)
- moved SERVO_LB0 8.89 mm to (185.4, 148.6)
- moved SERVO_LB2 8.89 mm to (185.4, 158.8)
- moved SERVO_RB0 8.89 mm to (259.1, 148.6)
- moved SERVO_RB2 8.89 mm to (259.1, 158.8)
- moved C4 6.84 mm to (185.4, 170.2), turned to 270 degrees
- moved C3 6.84 mm to (259.1, 170.2), turned to 270 degrees
- moved C1 3.81 mm to (256.5, 115.6)
- moved C2 3.81 mm to (188.0, 115.6)
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Connections:
- ALIM_BOARD1 pad 2: /ALIM/BAT -> N-0000080
- POW_BATTERY1 pad 2: N-0000080 -> /ALIM/BAT
- SECURITY_SWITCH1 pad 1: N-0000080 -> /ALIM/BAT
- SECURITY_SWITCH1 pad 2: /ALIM/BAT -> N-0000080
Routing:
- net /ALIM/POW_5V: track 262.0 -> 238.1 mm, vias 0 -> 1
- net /ARDUINO/LOG_5V: track 103.4 -> 117.0 mm
- net /ARDUINO/SCL: track 67.8 -> 79.8 mm
- net /LEG_RB/PWM0: track 45.1 -> 35.4 mm
- net /LEG_LB/PWM1: track 34.5 -> 43.4 mm
- net /LEG_LB/PWM0: track 37.4 -> 46.3 mm
- net /LEG_RB/PWM2: track 46.9 -> 38.0 mm
- net /LEG_RB/PWM1: track 44.3 -> 36.2 mm
- net /LEG_LF/PWM1: track 67.3 -> 59.9 mm
- net /LEG_LF/PWM0: track 68.3 -> 60.9 mm
- net /LEG_LF/PWM2: track 68.3 -> 60.9 mm
- net /ALIM/BAT: track 27.3 -> 20.1 mm
- net /LEG_LB/PWM2: track 40.6 -> 47.3 mm
- net N-0000080: track 23.5 -> 18.8 mm
- net /ARDUINO/SDA: track 63.5 -> 65.8 mm
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Other:
- net class Default: clearance 0.25 -> 0.1; via_dia 0.89 -> 0.889
- rule trace_clearance: 0.25 -> 0.1
