File: elec/adm_shield/adm_shield.sch (KiCad schematic (older format))
At the start: 0 parts

Commit message: Begining of the PCB.
Changed lines of the file:
@@
 $Sheet
 S 7900 1450 550  850
-U 54F0EBC1
+U 54F1C80B
 F0 "LEG_RF" 50
 F1 "leg.sch" 50
@@
 $Sheet
 S 2300 5700 550  850
-U 54F0EBC1
+U 54F1C80A
 F0 "LEG_LB" 50
 F1 "leg.sch" 50
@@
 $Sheet
 S 7950 5700 550  850
-U 54F0EBC1
+U 54F1C809
 F0 "LEG_RB" 50
 F1 "leg.sch" 50
@@
 Wire Wire Line
 	4800 2750 4700 2750
+Text Label 4700 2900 2    60   ~ 0
+LOG
 Text Label 4700 2750 2    60   ~ 0
-LOG
-Text Label 4700 2900 2    60   ~ 0
 GND
 $EndSCHEMATC
