File: elec/adm_shield/alim.sch (KiCad schematic (older format))
At the start: 4 parts

Commit message: Schematics finished ?
Parts:
- removed PULL_DOWN_2.7kOhm: R, ~, symbol R
- added ENABLE_ALIM: CONN_1, ~, symbol CONN_1
Connections:
- net at ALIM_BOARD.1: now also ENABLE_ALIM.1; no longer SECURITY_SWITCH.2
- net at ALIM_BOARD.2: now also SECURITY_SWITCH.2; no longer POW_BATTERY.2 (PM)
- net EN: no longer names the net of SECURITY_SWITCH.1
- net EN: now also POW_BATTERY.2 (PM)
Other:
- moved on the sheet: POW_BATTERY, SECURITY_SWITCH
Changed lines of the file:
@@
 $Descr A4 11693 8268
 encoding utf-8
-Sheet 20 20
+Sheet 15 24
 Title ""
-Date "27 feb 2015"
+Date "28 feb 2015"
 Rev ""
 Comp ""
@@
 	1    0    0    -1
 $EndComp
-Text HLabel 4500 3750 3    60   Input ~ 0
+Text HLabel 4250 3950 0    60   Input ~ 0
 GND
-Text HLabel 5700 3600 0    60   Input ~ 0
+Text HLabel 4250 4100 0    60   Input ~ 0
 POW_5V
-Text HLabel 4550 3200 0    60   Input ~ 0
-EN
-Text HLabel 4550 2900 0    60   Input ~ 0
-GND
-$Comp
-L R PULL_DOWN_2.7kOhm
-U 1 1 54F28DA2
-P 4800 2900
-F 0 "PULL_DOWN_2.7kOhm" V 4880 2900 40  0000 C CNN
-F 1 "R" V 4807 2901 40  0000 C CNN
-F 2 "~" V 4730 2900 30  0000 C CNN
-F 3 "~" H 4800 2900 30  0000 C CNN
-	1    4800 2900
-	0    -1   -1   0
-$EndComp
 $Comp
 L SW_PUSH SECURITY_SWITCH
 U 1 1 54F28DC0
-P 4850 3200
-F 0 "SECURITY_SWITCH" H 5000 3310 50  0000 C CNN
-F 1 "SW_PUSH" H 4850 3120 50  0000 C CNN
-F 2 "~" H 4850 3200 60  0000 C CNN
-F 3 "~" H 4850 3200 60  0000 C CNN
-	1    4850 3200
+P 4550 3550
+F 0 "SECURITY_SWITCH" H 4550 3650 50  0000 C CNN
+F 1 "SW_PUSH" H 4550 3470 50  0000 C CNN
+F 2 "~" H 4550 3550 60  0000 C CNN
+F 3 "~" H 4550 3550 60  0000 C CNN
+	1    4550 3550
 	1    0    0    -1
 $EndComp
-Wire Wire Line
-	5050 2900 5150 2900
-Wire Wire Line
-	5150 2900 5150 3200
-Wire Wire Line
-	5150 3200 5700 3200
 $Comp
 L CONN_2 POW_BATTERY
 U 1 1 54F28DD3
-P 4150 3650
-F 0 "POW_BATTERY" V 4100 3650 40  0000 C CNN
-F 1 "CONN_2" V 4200 3650 40  0000 C CNN
-F 2 "~" H 4150 3650 60  0000 C CNN
-F 3 "~" H 4150 3650 60  0000 C CNN
-	1    4150 3650
+P 3900 3650
+F 0 "POW_BATTERY" V 3850 3650 40  0000 C CNN
+F 1 "CONN_2" V 3950 3650 40  0000 C CNN
+F 2 "~" H 3900 3650 60  0000 C CNN
+F 3 "~" H 3900 3650 60  0000 C CNN
+	1    3900 3650
 	-1   0    0    1
 $EndComp
 Wire Wire Line
-	4500 3550 5150 3550
+	4950 3300 5700 3300
 Wire Wire Line
-	5150 3550 5150 3300
+	4950 3300 4950 3550
 Wire Wire Line
-	5150 3300 5700 3300
+	4950 3550 4850 3550
 Wire Wire Line
-	4500 3750 5250 3750
+	4250 3750 5150 3750
 Wire Wire Line
-	5600 3400 5600 3500
+	5150 3750 5150 3400
 Wire Wire Line
-	5600 3500 5700 3500
-Connection ~ 5600 3400
+	5150 3400 5700 3400
 Wire Wire Line
-	5250 3750 5250 3400
-Connection ~ 5250 3400
+	5550 3400 5550 3500
 Wire Wire Line
-	5250 3400 5700 3400
+	5550 3500 5700 3500
+Connection ~ 5550 3400
+Wire Wire Line
+	4400 3750 4400 3950
+Wire Wire Line
+	4400 3950 4250 3950
+Connection ~ 4400 3750
+Wire Wire Line
+	5700 3600 5350 3600
+Wire Wire Line
+	5350 3600 5350 4100
+Wire Wire Line
+	5350 4100 4250 4100
+$Comp
+L CONN_1 ENABLE_ALIM
+U 1 1 54F2D645
+P 4100 3200
+F 0 "ENABLE_ALIM" H 4180 3200 40  0000 L CNN
+F 1 "CONN_1" H 4100 3255 30  0001 C CNN
+F 2 "~" H 4100 3200 60  0000 C CNN
+F 3 "~" H 4100 3200 60  0000 C CNN
+	1    4100 3200
+	-1   0    0    1
+$EndComp
+Wire Wire Line
+	4250 3200 5700 3200
 $EndSCHEMATC

Commit message: Begining of the PCB.
Parts:
- renumbered ALIM_BOARD to ALIM_BOARD1, ENABLE_ALIM to ENABLE_ALIM1, POW_BATTERY to POW_BATTERY1, SECURITY_SWITCH to SECURITY_SWITCH1
Changed lines of the file:
@@
 $Descr A4 11693 8268
 encoding utf-8
-Sheet 15 24
+Sheet 14 24
 Title ""
 Date "28 feb 2015"
@@
 $EndDescr
 $Comp
-L CONN_5 ALIM_BOARD
+L CONN_5 ALIM_BOARD1
 U 1 1 54F28D93
 P 6100 3400
-F 0 "ALIM_BOARD" V 6050 3400 50  0000 C CNN
+F 0 "ALIM_BOARD1" V 6050 3400 50  0000 C CNN
 F 1 "CONN_5" V 6150 3400 50  0000 C CNN
 F 2 "~" H 6100 3400 60  0000 C CNN
@@
 POW_5V
 $Comp
-L SW_PUSH SECURITY_SWITCH
+L SW_PUSH SECURITY_SWITCH1
 U 1 1 54F28DC0
 P 4550 3550
-F 0 "SECURITY_SWITCH" H 4550 3650 50  0000 C CNN
+F 0 "SECURITY_SWITCH1" H 4550 3650 50  0000 C CNN
 F 1 "SW_PUSH" H 4550 3470 50  0000 C CNN
 F 2 "~" H 4550 3550 60  0000 C CNN
@@
 $EndComp
 $Comp
-L CONN_2 POW_BATTERY
+L CONN_2 POW_BATTERY1
 U 1 1 54F28DD3
 P 3900 3650
-F 0 "POW_BATTERY" V 3850 3650 40  0000 C CNN
+F 0 "POW_BATTERY1" V 3850 3650 40  0000 C CNN
 F 1 "CONN_2" V 3950 3650 40  0000 C CNN
 F 2 "~" H 3900 3650 60  0000 C CNN
@@
 	5350 4100 4250 4100
 $Comp
-L CONN_1 ENABLE_ALIM
+L CONN_1 ENABLE_ALIM1
 U 1 1 54F2D645
 P 4100 3200
-F 0 "ENABLE_ALIM" H 4180 3200 40  0000 L CNN
+F 0 "ENABLE_ALIM1" H 4180 3200 40  0000 L CNN
 F 1 "CONN_1" H 4100 3255 30  0001 C CNN
 F 2 "~" H 4100 3200 60  0000 C CNN

Commit message: Shield V2 (PCB begining)
Connections:
- net EN: now reaches ALIM_BOARD1.1, ENABLE_ALIM1.1
- net BAT: now reaches ALIM_BOARD1.2, SECURITY_SWITCH1.2
Changed lines of the file:
@@
 Sheet 14 24
 Title ""
-Date "28 feb 2015"
+Date "1 mar 2015"
 Rev ""
 Comp ""
@@
 Wire Wire Line
 	4250 3200 5700 3200
+Text Label 4950 3300 2    60   ~ 0
+BAT
+Text Label 4250 3050 2    60   ~ 0
+EN
+Wire Wire Line
+	4350 3200 4350 3050
+Wire Wire Line
+	4350 3050 4250 3050
+Connection ~ 4350 3200
 $EndSCHEMATC

Commit message: V3.1 ?
Parts:
- added C5: C, ~, symbol C
Connections:
- net BAT: now also POW_BATTERY1.2 (PM), SECURITY_SWITCH1.1, C5.1; no longer ALIM_BOARD1.2, SECURITY_SWITCH1.2
- net GND: now also C5.2
- new net: ALIM_BOARD1.2, SECURITY_SWITCH1.2
Other:
- moved on the sheet: ENABLE_ALIM1, SECURITY_SWITCH1
Changed lines of the file:
@@
 Sheet 14 24
 Title ""
-Date "1 mar 2015"
+Date "2 mar 2015"
 Rev ""
 Comp ""
@@
 L SW_PUSH SECURITY_SWITCH1
 U 1 1 54F28DC0
-P 4550 3550
-F 0 "SECURITY_SWITCH1" H 4550 3650 50  0000 C CNN
-F 1 "SW_PUSH" H 4550 3470 50  0000 C CNN
-F 2 "~" H 4550 3550 60  0000 C CNN
-F 3 "~" H 4550 3550 60  0000 C CNN
-	1    4550 3550
+P 4850 3300
+F 0 "SECURITY_SWITCH1" H 4850 3400 50  0000 C CNN
+F 1 "SW_PUSH" H 4850 3220 50  0000 C CNN
+F 2 "~" H 4850 3300 60  0000 C CNN
+F 3 "~" H 4850 3300 60  0000 C CNN
+	1    4850 3300
 	1    0    0    -1
 $EndComp
@@
 	-1   0    0    1
 $EndComp
-Wire Wire Line
-	4950 3300 5700 3300
-Wire Wire Line
-	4950 3300 4950 3550
-Wire Wire Line
-	4950 3550 4850 3550
+$Comp
+L CONN_1 ENABLE_ALIM1
+U 1 1 54F2D645
+P 5550 3200
+F 0 "ENABLE_ALIM1" H 5350 3250 40  0000 L CNN
+F 1 "CONN_1" H 5550 3255 30  0001 C CNN
+F 2 "~" H 5550 3200 60  0000 C CNN
+F 3 "~" H 5550 3200 60  0000 C CNN
+	1    5550 3200
+	-1   0    0    1
+$EndComp
+Text Label 5700 3200 2    60   ~ 0
+EN
+$Comp
+L C C5
+U 1 1 54F4629D
+P 4400 3500
+F 0 "C5" H 4400 3600 40  0000 L CNN
+F 1 "C" H 4406 3415 40  0000 L CNN
+F 2 "~" H 4438 3350 30  0000 C CNN
+F 3 "~" H 4400 3500 60  0000 C CNN
+	1    4400 3500
+	1    0    0    -1
+$EndComp
 Wire Wire Line
 	4250 3750 5150 3750
-Wire Wire Line
-	5150 3750 5150 3400
 Wire Wire Line
 	5150 3400 5700 3400
@@
 Connection ~ 5550 3400
 Wire Wire Line
-	4400 3750 4400 3950
+	4400 3700 4400 3950
 Wire Wire Line
 	4400 3950 4250 3950
@@
 Wire Wire Line
 	5350 4100 4250 4100
-$Comp
-L CONN_1 ENABLE_ALIM1
-U 1 1 54F2D645
-P 4100 3200
-F 0 "ENABLE_ALIM1" H 4180 3200 40  0000 L CNN
-F 1 "CONN_1" H 4100 3255 30  0001 C CNN
-F 2 "~" H 4100 3200 60  0000 C CNN
-F 3 "~" H 4100 3200 60  0000 C CNN
-	1    4100 3200
-	-1   0    0    1
-$EndComp
+Text Label 4400 3300 2    60   ~ 0
+BAT
 Wire Wire Line
-	4250 3200 5700 3200
-Text Label 4950 3300 2    60   ~ 0
-BAT
-Text Label 4250 3050 2    60   ~ 0
-EN
+	4250 3550 4250 3300
 Wire Wire Line
-	4350 3200 4350 3050
+	4250 3300 4550 3300
+Connection ~ 4400 3300
 Wire Wire Line
-	4350 3050 4250 3050
-Connection ~ 4350 3200
+	5150 3300 5700 3300
+Wire Wire Line
+	5150 3750 5150 3400
 $EndSCHEMATC
