File: elec/adm_shield/arduino.sch (KiCad schematic (older format))
At the start: 1 part

Commit message: Schematics finished ?
Connections:
- net GP2_LB: now also SHIELD?.AD11; no longer SHIELD?.AD3
- net GP2_LF: now also SHIELD?.AD8; no longer SHIELD?.AD0
- net GP2_RB: now also SHIELD?.AD10; no longer SHIELD?.AD2
- net GP2_RF: now also SHIELD?.AD9; no longer SHIELD?.AD1
- net SS4: now reaches SHIELD?.34 (PC3)
- net SENS_0: now reaches SHIELD?.AD12
- net SENS_1: now reaches SHIELD?.AD13
- net SENS_2: now reaches SHIELD?.AD14
- net SENS_3: now reaches SHIELD?.AD15
Changed lines of the file:
@@
 $Descr A4 11693 8268
 encoding utf-8
-Sheet 18 20
+Sheet 20 24
 Title ""
-Date "27 feb 2015"
+Date "28 feb 2015"
 Rev ""
 Comp ""
@@
 Text HLabel 6450 3700 2    60   Input ~ 0
 SDA
-Text HLabel 4550 2400 0    60   Input ~ 0
+Text HLabel 4550 3300 0    60   Input ~ 0
 GP2_LF
-Text HLabel 4550 2500 0    60   Input ~ 0
+Text HLabel 4550 3400 0    60   Input ~ 0
 GP2_RF
-Text HLabel 4550 2600 0    60   Input ~ 0
+Text HLabel 4550 3500 0    60   Input ~ 0
 GP2_RB
-Text HLabel 4550 2700 0    60   Input ~ 0
+Text HLabel 4550 3600 0    60   Input ~ 0
 GP2_LB
 Text HLabel 6450 3600 2    60   Input ~ 0
@@
 Text HLabel 6450 5650 2    60   Input ~ 0
 SS3
+Text HLabel 6450 5550 2    60   Input ~ 0
+SS4
+Text HLabel 4550 3700 0    60   Input ~ 0
+SENS_0
+Text HLabel 4550 3800 0    60   Input ~ 0
+SENS_1
+Text HLabel 4550 3900 0    60   Input ~ 0
+SENS_2
+Text HLabel 4550 4000 0    60   Input ~ 0
+SENS_3
 $EndSCHEMATC

Commit message: Begining of the PCB.
Parts:
- gave numbers to parts that had none: 1
Changed lines of the file:
@@
 $Descr A4 11693 8268
 encoding utf-8
-Sheet 20 24
+Sheet 19 24
 Title ""
 Date "28 feb 2015"
@@
 $EndDescr
 $Comp
-L ARDUINO_MEGA_SHIELD SHIELD?
+L ARDUINO_MEGA_SHIELD SHIELD1
 U 1 1 54F159EE
 P 5550 3650
-F 0 "SHIELD?" H 5150 6150 60  0000 C CNN
+F 0 "SHIELD1" H 5150 6150 60  0000 C CNN
 F 1 "ARDUINO_MEGA_SHIELD" H 5450 950 60  0000 C CNN
 F 2 "" H 5550 3650 60  0000 C CNN

Commit message: PCB almost finished ?
Connections:
- net PWM_LB0: now also SHIELD1.47 (PL2)
- net PWM_LB2: now also SHIELD1.43 (PL6)
Changed lines of the file:
@@
 Text HLabel 6450 2000 2    60   Input ~ 0
 PWM_RB2
-Text HLabel 4550 5250 0    60   Input ~ 0
+Text HLabel 4500 5250 0    60   Input ~ 0
 PWM_LB0
 Text HLabel 4550 5350 0    60   Input ~ 0
 PWM_LB1
-Text HLabel 4550 5450 0    60   Input ~ 0
+Text HLabel 4500 5450 0    60   Input ~ 0
 PWM_LB2
 Text HLabel 4550 1900 0    60   Input ~ 0
@@
 Text HLabel 4550 4000 0    60   Input ~ 0
 SENS_3
+Wire Wire Line
+	4550 5250 4500 5250
+Wire Wire Line
+	4550 5150 4500 5150
+Wire Wire Line
+	4500 5150 4500 5250
+Wire Wire Line
+	4550 5450 4500 5450
+Wire Wire Line
+	4550 5550 4500 5550
+Wire Wire Line
+	4500 5550 4500 5450
 $EndSCHEMATC

Commit message: First version PCB.
Connections:
- net LOG_5V: no longer SHIELD1.5V_4, SHIELD1.5V_5
Changed lines of the file:
@@
 Text HLabel 4550 1900 0    60   Input ~ 0
-LOG_5V
-Text HLabel 6450 4050 2    60   Input ~ 0
-LOG_5V
-Text HLabel 6450 4150 2    60   Input ~ 0
 LOG_5V
 Text HLabel 4550 2000 0    60   Input ~ 0

Commit message: Shield V2 (PCB begining)
Connections:
- net PWM_RB0: now also SHIELD1.5; no longer SHIELD1.6
- net PWM_RB1: now also SHIELD1.3; no longer SHIELD1.7
- net PWM_RB2: now also SHIELD1.2; no longer SHIELD1.8
- net PWM_RF0: now also SHIELD1.6; no longer SHIELD1.5
- net PWM_RF1: now also SHIELD1.7; no longer SHIELD1.2
- net PWM_RF2: now also SHIELD1.8; no longer SHIELD1.3
Changed lines of the file:
@@
 Sheet 19 24
 Title ""
-Date "28 feb 2015"
+Date "1 mar 2015"
 Rev ""
 Comp ""
@@
 Text HLabel 6450 1500 2    60   Input ~ 0
 PWM_LF2
+Text HLabel 6450 2300 2    60   Input ~ 0
+PWM_RF0
+Text HLabel 6450 2200 2    60   Input ~ 0
+PWM_RF1
+Text HLabel 6450 2000 2    60   Input ~ 0
+PWM_RF2
 Text HLabel 6450 2400 2    60   Input ~ 0
-PWM_RF0
+PWM_RB0
+Text HLabel 6450 2600 2    60   Input ~ 0
+PWM_RB1
 Text HLabel 6450 2700 2    60   Input ~ 0
-PWM_RF1
-Text HLabel 6450 2600 2    60   Input ~ 0
-PWM_RF2
-Text HLabel 6450 2300 2    60   Input ~ 0
-PWM_RB0
-Text HLabel 6450 2200 2    60   Input ~ 0
-PWM_RB1
-Text HLabel 6450 2000 2    60   Input ~ 0
 PWM_RB2
 Text HLabel 4500 5250 0    60   Input ~ 0

Commit message: PCB FINISHED ! + Correction of schematics.
Connections:
- net GND: no longer SHIELD1.GND1
Changed lines of the file:
@@
 Text HLabel 4550 1900 0    60   Input ~ 0
 LOG_5V
-Text HLabel 4550 2000 0    60   Input ~ 0
-GND
 Text HLabel 4550 2100 0    60   Input ~ 0
 GND
