File: elec/adm_shield/gp2.sch (KiCad schematic (older format))
At the start: 4 parts

Commit message: Begining of the PCB.
Parts:
- renumbered GP2_LB to GP2_LB1, GP2_LF to GP2_LF1, GP2_RB to GP2_RB1, GP2_RF to GP2_RF1
Changed lines of the file:
@@
 $Descr User 7874 4000
 encoding utf-8
-Sheet 22 24
+Sheet 20 24
 Title ""
 Date "28 feb 2015"
@@
 $EndDescr
 $Comp
-L CONN_3 GP2_LF
+L CONN_3 GP2_LF1
 U 1 1 54F33CA3
 P 3050 1400
-F 0 "GP2_LF" V 3000 1400 50  0000 C CNN
+F 0 "GP2_LF1" V 3000 1400 50  0000 C CNN
 F 1 "CONN_3" V 3100 1400 40  0000 C CNN
 F 2 "~" H 3050 1400 60  0000 C CNN
@@
 LOG_5V
 $Comp
-L CONN_3 GP2_RF
+L CONN_3 GP2_RF1
 U 1 1 54F33D31
 P 3550 1400
-F 0 "GP2_RF" V 3500 1400 50  0000 C CNN
+F 0 "GP2_RF1" V 3500 1400 50  0000 C CNN
 F 1 "CONN_3" V 3600 1400 40  0000 C CNN
 F 2 "~" H 3550 1400 60  0000 C CNN
@@
 LOG_5V
 $Comp
-L CONN_3 GP2_RB
+L CONN_3 GP2_RB1
 U 1 1 54F33D39
 P 4050 1400
-F 0 "GP2_RB" V 4000 1400 50  0000 C CNN
+F 0 "GP2_RB1" V 4000 1400 50  0000 C CNN
 F 1 "CONN_3" V 4100 1400 40  0000 C CNN
 F 2 "~" H 4050 1400 60  0000 C CNN
@@
 LOG_5V
 $Comp
-L CONN_3 GP2_LB
+L CONN_3 GP2_LB1
 U 1 1 54F33D41
 P 4550 1400
-F 0 "GP2_LB" V 4500 1400 50  0000 C CNN
+F 0 "GP2_LB1" V 4500 1400 50  0000 C CNN
 F 1 "CONN_3" V 4600 1400 40  0000 C CNN
 F 2 "~" H 4550 1400 60  0000 C CNN

Commit message: Shield V2 (PCB begining)
Connections:
- net GND: now also GP2_LB1.1 (P1), GP2_LF1.1 (P1), GP2_RB1.1 (P1), GP2_RF1.1 (P1); no longer GP2_LB1.3 (P3), GP2_LF1.3 (P3), GP2_RB1.3 (P3), GP2_RF1.3 (P3)
- net GP2_LB: now also GP2_LB1.3 (P3); no longer GP2_LB1.1 (P1)
- net GP2_LF: now also GP2_LF1.3 (P3); no longer GP2_LF1.1 (P1)
- net GP2_RB: now also GP2_RB1.3 (P3); no longer GP2_RB1.1 (P1)
- net GP2_RF: now also GP2_RF1.3 (P3); no longer GP2_RF1.1 (P1)
Changed lines of the file:
@@
 Sheet 20 24
 Title ""
-Date "28 feb 2015"
+Date "1 mar 2015"
 Rev ""
 Comp ""
@@
 	0    -1   -1   0
 $EndComp
-Text HLabel 3150 1750 3    60   Input ~ 0
+Text HLabel 2950 1750 3    60   Input ~ 0
 GND
 Text HLabel 3050 1750 3    60   Input ~ 0
@@
 	0    -1   -1   0
 $EndComp
-Text HLabel 3650 1750 3    60   Input ~ 0
+Text HLabel 3450 1750 3    60   Input ~ 0
 GND
 Text HLabel 3550 1750 3    60   Input ~ 0
@@
 	0    -1   -1   0
 $EndComp
-Text HLabel 4150 1750 3    60   Input ~ 0
+Text HLabel 3950 1750 3    60   Input ~ 0
 GND
 Text HLabel 4050 1750 3    60   Input ~ 0
@@
 	0    -1   -1   0
 $EndComp
-Text HLabel 4650 1750 3    60   Input ~ 0
+Text HLabel 4450 1750 3    60   Input ~ 0
 GND
 Text HLabel 4550 1750 3    60   Input ~ 0
 LOG_5V
-Text HLabel 2950 1750 3    60   Input ~ 0
+Text HLabel 3150 1750 3    60   Input ~ 0
 GP2_LF
-Text HLabel 3450 1750 3    60   Input ~ 0
+Text HLabel 3650 1750 3    60   Input ~ 0
 GP2_RF
-Text HLabel 3950 1750 3    60   Input ~ 0
+Text HLabel 4150 1750 3    60   Input ~ 0
 GP2_RB
-Text HLabel 4450 1750 3    60   Input ~ 0
+Text HLabel 4650 1750 3    60   Input ~ 0
 GP2_LB
 $EndSCHEMATC
