File: elec/adm_shield/gpio.sch (KiCad schematic (older format))
At the start: 1 part

Commit message: Begining of the PCB.
Parts:
- renumbered GPIO to GPIO1
Connections:
- net GPIO0: now also GPIO1.3; no longer GPIO1.2
- net GPIO1: now also GPIO1.4; no longer GPIO1.3
- net GPIO2: now also GPIO1.5; no longer GPIO1.4
- net GPIO3: now also GPIO1.6; no longer GPIO1.5
- net LOG_5V: now also GPIO1.2; no longer GPIO1.6
Changed lines of the file:
@@
 $Descr User 5197 4000
 encoding utf-8
-Sheet 23 24
+Sheet 21 24
 Title ""
 Date "28 feb 2015"
@@
 $EndDescr
 $Comp
-L CONN_6 GPIO
+L CONN_6 GPIO1
 U 1 1 54F37CAA
 P 2700 1700
-F 0 "GPIO" V 2650 1700 60  0000 C CNN
+F 0 "GPIO1" V 2650 1700 60  0000 C CNN
 F 1 "CONN_6" V 2750 1700 60  0000 C CNN
 F 2 "~" H 2700 1700 60  0000 C CNN
@@
 Text HLabel 2350 1450 0    60   Input ~ 0
 GND
+Text HLabel 2350 1550 0    60   Input ~ 0
+LOG_5V
+Text HLabel 2350 1650 0    60   Input ~ 0
+GPIO0
+Text HLabel 2350 1750 0    60   Input ~ 0
+GPIO1
+Text HLabel 2350 1850 0    60   Input ~ 0
+GPIO2
 Text HLabel 2350 1950 0    60   Input ~ 0
-LOG_5V
-Text HLabel 2350 1550 0    60   Input ~ 0
-GPIO0
-Text HLabel 2350 1650 0    60   Input ~ 0
-GPIO1
-Text HLabel 2350 1750 0    60   Input ~ 0
-GPIO2
-Text HLabel 2350 1850 0    60   Input ~ 0
 GPIO3
 $EndSCHEMATC
