File: elec/adm_shield/leg.sch (KiCad schematic (older format))
At the start: 0 parts

Commit message: Shield V2 (PCB begining)
Parts:
- added C1: C, ~, symbol C
Connections:
- net GND: now also C1.2
- net POW_5V: now also C1.1
Changed lines of the file:
@@
 $Descr A4 11693 8268
 encoding utf-8
-Sheet 10 24
+Sheet 2 24
 Title ""
-Date "28 feb 2015"
+Date "1 mar 2015"
 Rev ""
 Comp ""
@@
 $EndDescr
 $Sheet
-S 3550 4000 800  650
+S 3550 2950 800  650
 U 54F06B67
 F0 "SERVO1" 50
+F1 "servo.sch" 50
+F2 "GND" I R 4350 3450 60
+F3 "PWM" I R 4350 3050 60
+F4 "POW_5V" I R 4350 3250 60
+$EndSheet
+$Sheet
+S 3550 4000 800  650
+U 54F1C808
+F0 "SERVO2" 50
 F1 "servo.sch" 50
 F2 "GND" I R 4350 4500 60
 F3 "PWM" I R 4350 4100 60
 F4 "POW_5V" I R 4350 4300 60
-$EndSheet
-$Sheet
-S 3550 2950 800  650
-U 54F1C808
-F0 "SERVO2" 50
-F1 "servo.sch" 50
-F2 "GND" I R 4350 3450 60
-F3 "PWM" I R 4350 3050 60
-F4 "POW_5V" I R 4350 3250 60
 $EndSheet
 $Sheet
@@
 Text HLabel 4350 2150 2    60   Input ~ 0
 POW_5V
+$Comp
+L C C1
+U 1 1 54F2D541
+P 6050 2400
+AR Path="/54F0EBC1/54F2D541" Ref="C1"  Part="1"
+AR Path="/54F1C80B/54F2D541" Ref="C2"  Part="1"
+AR Path="/54F1C80A/54F2D541" Ref="C3"  Part="1"
+AR Path="/54F1C809/54F2D541" Ref="C4"  Part="1"
+F 0 "C1" H 6050 2500 40  0000 L CNN
+F 1 "C" H 6056 2315 40  0000 L CNN
+F 2 "~" H 6088 2250 30  0000 C CNN
+F 3 "~" H 6050 2400 60  0000 C CNN
+	1    6050 2400
+	-1   0    0    1
+$EndComp
+Text HLabel 6200 2600 2    60   Input ~ 0
+POW_5V
+Text HLabel 6200 2200 2    60   Input ~ 0
+GND
+Wire Wire Line
+	6050 2200 6200 2200
+Wire Wire Line
+	6050 2600 6200 2600
 $EndSCHEMATC

Commit message: PCB FINISHED ! + Correction of schematics.
Changed lines of the file:
@@
 AR Path="/54F1C80A/54F2D541" Ref="C3"  Part="1"
 AR Path="/54F1C809/54F2D541" Ref="C4"  Part="1"
-F 0 "C1" H 6050 2500 40  0000 L CNN
+F 0 "C3" H 6050 2500 40  0000 L CNN
 F 1 "C" H 6056 2315 40  0000 L CNN
 F 2 "~" H 6088 2250 30  0000 C CNN

Commit message: V3.1 ?
Changed lines of the file:
@@
 Sheet 2 24
 Title ""
-Date "1 mar 2015"
+Date "2 mar 2015"
 Rev ""
 Comp ""
@@
 AR Path="/54F1C80A/54F2D541" Ref="C3"  Part="1"
 AR Path="/54F1C809/54F2D541" Ref="C4"  Part="1"
-F 0 "C3" H 6050 2500 40  0000 L CNN
+F 0 "C4" H 6050 2500 40  0000 L CNN
 F 1 "C" H 6056 2315 40  0000 L CNN
 F 2 "~" H 6088 2250 30  0000 C CNN
