File: elec/adm_shield/servo.sch (KiCad schematic (older format))
At the start: 2 parts

Commit message: Schematics finished ?
Parts:
- gave numbers to parts that had none: 1
Changed lines of the file:
@@
 $Descr A4 11693 8268
 encoding utf-8
-Sheet 2 20
+Sheet 3 24
 Title ""
-Date "27 feb 2015"
+Date "28 feb 2015"
 Rev ""
 Comp ""
@@
 $EndDescr
 $Comp
-L CONN_3 K?
+L CONN_3 SERVO?
 U 1 1 54F06C2D
 P 7100 3500
-F 0 "K?" V 7050 3500 50  0000 C CNN
+F 0 "SERVO?" V 7050 3500 50  0000 C CNN
 F 1 "CONN_3" V 7150 3500 40  0000 C CNN
 F 2 "" H 7100 3500 60  0000 C CNN

Commit message: Begining of the PCB.
Parts:
- gave numbers to parts that had none: 2
Changed lines of the file:
@@
 $Descr A4 11693 8268
 encoding utf-8
-Sheet 3 24
+Sheet 13 24
 Title ""
 Date "28 feb 2015"
@@
 $EndDescr
 $Comp
-L CONN_3 SERVO?
+L CONN_3 SERVO_LF1
 U 1 1 54F06C2D
 P 7100 3500
-F 0 "SERVO?" V 7050 3500 50  0000 C CNN
+AR Path="/54F0EBC1/54F06B67/54F06C2D" Ref="SERVO_LF1"  Part="1"
+AR Path="/54F0EBC1/54F1C808/54F06C2D" Ref="SERVO_LF2"  Part="1"
+AR Path="/54F0EBC1/54F1C807/54F06C2D" Ref="SERVO_LF0"  Part="1"
+AR Path="/54F1C80B/54F06B67/54F06C2D" Ref="SERVO_RF2"  Part="1"
+AR Path="/54F1C80B/54F1C808/54F06C2D" Ref="SERVO_RF1"  Part="1"
+AR Path="/54F1C80B/54F1C807/54F06C2D" Ref="SERVO_RF0"  Part="1"
+AR Path="/54F1C80A/54F06B67/54F06C2D" Ref="SERVO_RB1"  Part="1"
+AR Path="/54F1C80A/54F1C808/54F06C2D" Ref="SERVO_RB2"  Part="1"
+AR Path="/54F1C80A/54F1C807/54F06C2D" Ref="SERVO_RB0"  Part="1"
+AR Path="/54F1C809/54F06B67/54F06C2D" Ref="SERVO_LB1"  Part="1"
+AR Path="/54F1C809/54F1C808/54F06C2D" Ref="SERVO_LB2"  Part="1"
+AR Path="/54F1C809/54F1C807/54F06C2D" Ref="SERVO_LB0"  Part="1"
+F 0 "SERVO_RB0" V 7050 3500 50  0000 C CNN
 F 1 "CONN_3" V 7150 3500 40  0000 C CNN
 F 2 "" H 7100 3500 60  0000 C CNN
@@
 PWM
 $Comp
-L C C?
+L C C1
 U 1 1 54F06CAD
 P 6050 3700
-F 0 "C?" H 6050 3800 40  0000 L CNN
+AR Path="/54F0EBC1/54F06B67/54F06CAD" Ref="C1"  Part="1"
+AR Path="/54F0EBC1/54F1C808/54F06CAD" Ref="C2"  Part="1"
+AR Path="/54F0EBC1/54F1C807/54F06CAD" Ref="C3"  Part="1"
+AR Path="/54F1C80B/54F06B67/54F06CAD" Ref="C4"  Part="1"
+AR Path="/54F1C80B/54F1C808/54F06CAD" Ref="C5"  Part="1"
+AR Path="/54F1C80B/54F1C807/54F06CAD" Ref="C6"  Part="1"
+AR Path="/54F1C80A/54F06B67/54F06CAD" Ref="C7"  Part="1"
+AR Path="/54F1C80A/54F1C808/54F06CAD" Ref="C8"  Part="1"
+AR Path="/54F1C80A/54F1C807/54F06CAD" Ref="C9"  Part="1"
+AR Path="/54F1C809/54F06B67/54F06CAD" Ref="C10"  Part="1"
+AR Path="/54F1C809/54F1C808/54F06CAD" Ref="C11"  Part="1"
+AR Path="/54F1C809/54F1C807/54F06CAD" Ref="C12"  Part="1"
+F 0 "C9" H 6050 3800 40  0000 L CNN
 F 1 "C" H 6056 3615 40  0000 L CNN
 F 2 "~" H 6088 3550 30  0000 C CNN

Commit message: PCB almost finished ?
Changed lines of the file:
@@
 AR Path="/54F1C809/54F1C808/54F06C2D" Ref="SERVO_LB2"  Part="1"
 AR Path="/54F1C809/54F1C807/54F06C2D" Ref="SERVO_LB0"  Part="1"
-F 0 "SERVO_RB0" V 7050 3500 50  0000 C CNN
+F 0 "SERVO_LF0" V 7050 3500 50  0000 C CNN
 F 1 "CONN_3" V 7150 3500 40  0000 C CNN
 F 2 "" H 7100 3500 60  0000 C CNN
@@
 AR Path="/54F1C809/54F1C808/54F06CAD" Ref="C11"  Part="1"
 AR Path="/54F1C809/54F1C807/54F06CAD" Ref="C12"  Part="1"
-F 0 "C9" H 6050 3800 40  0000 L CNN
+F 0 "C3" H 6050 3800 40  0000 L CNN
 F 1 "C" H 6056 3615 40  0000 L CNN
 F 2 "~" H 6088 3550 30  0000 C CNN

Commit message: Shield V2 (PCB begining)
Parts:
- removed C1: C, ~, symbol C
Connections:
- net GND: now also SERVO_LF1.1 (P1); no longer SERVO_LF1.3 (P3)
- net PWM: now also SERVO_LF1.3 (P3); no longer SERVO_LF1.1 (P1)
Changed lines of the file:
@@
 $Descr A4 11693 8268
 encoding utf-8
-Sheet 13 24
+Sheet 7 24
 Title ""
-Date "28 feb 2015"
+Date "1 mar 2015"
 Rev ""
 Comp ""
@@
 AR Path="/54F0EBC1/54F1C808/54F06C2D" Ref="SERVO_LF2"  Part="1"
 AR Path="/54F0EBC1/54F1C807/54F06C2D" Ref="SERVO_LF0"  Part="1"
-AR Path="/54F1C80B/54F06B67/54F06C2D" Ref="SERVO_RF2"  Part="1"
-AR Path="/54F1C80B/54F1C808/54F06C2D" Ref="SERVO_RF1"  Part="1"
+AR Path="/54F1C80B/54F06B67/54F06C2D" Ref="SERVO_RF1"  Part="1"
+AR Path="/54F1C80B/54F1C808/54F06C2D" Ref="SERVO_RF2"  Part="1"
 AR Path="/54F1C80B/54F1C807/54F06C2D" Ref="SERVO_RF0"  Part="1"
-AR Path="/54F1C80A/54F06B67/54F06C2D" Ref="SERVO_RB1"  Part="1"
-AR Path="/54F1C80A/54F1C808/54F06C2D" Ref="SERVO_RB2"  Part="1"
-AR Path="/54F1C80A/54F1C807/54F06C2D" Ref="SERVO_RB0"  Part="1"
-AR Path="/54F1C809/54F06B67/54F06C2D" Ref="SERVO_LB1"  Part="1"
-AR Path="/54F1C809/54F1C808/54F06C2D" Ref="SERVO_LB2"  Part="1"
-AR Path="/54F1C809/54F1C807/54F06C2D" Ref="SERVO_LB0"  Part="1"
-F 0 "SERVO_LF0" V 7050 3500 50  0000 C CNN
+AR Path="/54F1C80A/54F06B67/54F06C2D" Ref="SERVO_LB1"  Part="1"
+AR Path="/54F1C80A/54F1C808/54F06C2D" Ref="SERVO_LB2"  Part="1"
+AR Path="/54F1C80A/54F1C807/54F06C2D" Ref="SERVO_LB0"  Part="1"
+AR Path="/54F1C809/54F06B67/54F06C2D" Ref="SERVO_RB1"  Part="1"
+AR Path="/54F1C809/54F1C808/54F06C2D" Ref="SERVO_RB2"  Part="1"
+AR Path="/54F1C809/54F1C807/54F06C2D" Ref="SERVO_RB0"  Part="1"
+F 0 "SERVO_RF1" V 7050 3500 50  0000 C CNN
 F 1 "CONN_3" V 7150 3500 40  0000 C CNN
 F 2 "" H 7100 3500 60  0000 C CNN
@@
 	1    0    0    -1
 $EndComp
-Text HLabel 5250 3900 0    60   Input ~ 0
+Text HLabel 5250 3100 0    60   Input ~ 0
 GND
 Text HLabel 5250 3500 0    60   Input ~ 0
 POW_5V
-Text HLabel 5250 3100 0    60   Input ~ 0
+Text HLabel 5250 3900 0    60   Input ~ 0
 PWM
-$Comp
-L C C1
-U 1 1 54F06CAD
-P 6050 3700
-AR Path="/54F0EBC1/54F06B67/54F06CAD" Ref="C1"  Part="1"
-AR Path="/54F0EBC1/54F1C808/54F06CAD" Ref="C2"  Part="1"
-AR Path="/54F0EBC1/54F1C807/54F06CAD" Ref="C3"  Part="1"
-AR Path="/54F1C80B/54F06B67/54F06CAD" Ref="C4"  Part="1"
-AR Path="/54F1C80B/54F1C808/54F06CAD" Ref="C5"  Part="1"
-AR Path="/54F1C80B/54F1C807/54F06CAD" Ref="C6"  Part="1"
-AR Path="/54F1C80A/54F06B67/54F06CAD" Ref="C7"  Part="1"
-AR Path="/54F1C80A/54F1C808/54F06CAD" Ref="C8"  Part="1"
-AR Path="/54F1C80A/54F1C807/54F06CAD" Ref="C9"  Part="1"
-AR Path="/54F1C809/54F06B67/54F06CAD" Ref="C10"  Part="1"
-AR Path="/54F1C809/54F1C808/54F06CAD" Ref="C11"  Part="1"
-AR Path="/54F1C809/54F1C807/54F06CAD" Ref="C12"  Part="1"
-F 0 "C3" H 6050 3800 40  0000 L CNN
-F 1 "C" H 6056 3615 40  0000 L CNN
-F 2 "~" H 6088 3550 30  0000 C CNN
-F 3 "~" H 6050 3700 60  0000 C CNN
-	1    6050 3700
-	1    0    0    -1
-$EndComp
-Wire Wire Line
-	5250 3500 6750 3500
-Connection ~ 6050 3500
 Wire Wire Line
 	5250 3900 6750 3900
 Wire Wire Line
 	6750 3900 6750 3600
-Connection ~ 6050 3900
 Wire Wire Line
 	6750 3400 6750 3100
 Wire Wire Line
 	6750 3100 5250 3100
+Wire Wire Line
+	5250 3500 6750 3500
 $EndSCHEMATC

Commit message: V3.1 ?
Changed lines of the file:
@@
 Sheet 7 24
 Title ""
-Date "1 mar 2015"
+Date "2 mar 2015"
 Rev ""
 Comp ""
@@
 AR Path="/54F1C809/54F1C808/54F06C2D" Ref="SERVO_RB2"  Part="1"
 AR Path="/54F1C809/54F1C807/54F06C2D" Ref="SERVO_RB0"  Part="1"
-F 0 "SERVO_RF1" V 7050 3500 50  0000 C CNN
+F 0 "SERVO_RF0" V 7050 3500 50  0000 C CNN
 F 1 "CONN_3" V 7150 3500 40  0000 C CNN
 F 2 "" H 7100 3500 60  0000 C CNN
