File: elec/adm_shield/spi.sch (KiCad schematic (older format))
At the start: 1 part

Commit message: Begining of the PCB.
Parts:
- renumbered SPI to SPI1
Changed lines of the file:
@@
 $Descr A4 11693 8268
 encoding utf-8
-Sheet 21 24
+Sheet 24 24
 Title ""
 Date "28 feb 2015"
@@
 $EndDescr
 $Comp
-L CONN_5X2 SPI
+L CONN_5X2 SPI1
 U 1 1 54F2F47D
 P 5800 3100
-F 0 "SPI" H 5800 3400 60  0000 C CNN
+F 0 "SPI1" H 5800 3400 60  0000 C CNN
 F 1 "CONN_5X2" V 5800 3100 50  0000 C CNN
 F 2 "~" H 5800 3100 60  0000 C CNN

Commit message: Shield V2 (PCB begining)
Connections:
- net MISO: now also SPI1.6; no longer SPI1.10
- net MOSI: now also SPI1.4; no longer SPI1.8
- net SCK: now also SPI1.8; no longer SPI1.6
- net SS: now also SPI1.10; no longer SPI1.4
Changed lines of the file:
@@
 Sheet 24 24
 Title ""
-Date "28 feb 2015"
+Date "1 mar 2015"
 Rev ""
 Comp ""
@@
 Text HLabel 6200 2900 2    60   Input ~ 0
 GND
+Text HLabel 6200 3300 2    60   Input ~ 0
+SS
+Text HLabel 6200 3200 2    60   Input ~ 0
+SCK
 Text HLabel 6200 3000 2    60   Input ~ 0
-SS
+MOSI
 Text HLabel 6200 3100 2    60   Input ~ 0
-SCK
-Text HLabel 6200 3200 2    60   Input ~ 0
-MOSI
-Text HLabel 6200 3300 2    60   Input ~ 0
 MISO
 Text HLabel 5400 3000 0    60   Input ~ 0
