File: elec/adm_shield/uart.sch (KiCad schematic (older format))
At the start: 1 part

Commit message: Begining of the PCB.
Parts:
- renumbered UART to UART1
Changed lines of the file:
@@
 $Descr A4 11693 8268
 encoding utf-8
-Sheet 24 24
+Sheet 22 24
 Title ""
 Date "28 feb 2015"
@@
 $EndDescr
 $Comp
-L CONN_3 UART
+L CONN_3 UART1
 U 1 1 54F3C0D8
 P 6100 4100
-F 0 "UART" V 6050 4100 50  0000 C CNN
+F 0 "UART1" V 6050 4100 50  0000 C CNN
 F 1 "CONN_3" V 6150 4100 40  0000 C CNN
 F 2 "~" H 6100 4100 60  0000 C CNN

Commit message: Shield V2 (PCB begining)
Connections:
- net GND: now also UART1.1 (P1); no longer UART1.3 (P3)
- net RX: now also UART1.3 (P3); no longer UART1.1 (P1)
Changed lines of the file:
@@
 Sheet 22 24
 Title ""
-Date "28 feb 2015"
+Date "1 mar 2015"
 Rev ""
 Comp ""
@@
 	1    0    0    -1
 $EndComp
-Text HLabel 5750 4000 0    60   Input ~ 0
+Text HLabel 5750 4200 0    60   Input ~ 0
 RX
 Text HLabel 5750 4100 0    60   Input ~ 0
 TX
-Text HLabel 5750 4200 0    60   Input ~ 0
+Text HLabel 5750 4000 0    60   Input ~ 0
 GND
 $EndSCHEMATC
