File: elec/teensy_shield/angle_sensor.sch (KiCad schematic (older format))
At the start: 0 parts

Commit message: Completed new board schematics.
Parts:
- added K?: CONN_3, symbol CONN_3
Connections:
- net GND: now also K?.1 (P1)
- net OUT: now also K?.3 (P3)
- net Vin: now also K?.2 (PM)
Changed lines of the file:
@@
 LIBS:contrib
 LIBS:valves
+LIBS:arduino_shieldsNCL
+LIBS:teensy
+LIBS:pololu
+LIBS:teensy_shield-cache
 EELAYER 24 0
 EELAYER END
 $Descr A4 11693 8268
 encoding utf-8
-Sheet 5 26
+Sheet 8 34
 Title ""
 Date ""
@@
 Comment4 ""
 $EndDescr
-Text HLabel 5200 2850 0    60   Input ~ 0
+Text HLabel 5500 3100 0    60   Input ~ 0
 Vin
-Text HLabel 5100 3100 0    60   Input ~ 0
+Text HLabel 5500 3000 0    60   Input ~ 0
 GND
-Text HLabel 5200 3350 0    60   Input ~ 0
+Text HLabel 5500 3200 0    60   Input ~ 0
 OUT
+$Comp
+L CONN_3 K?
+U 1 1 55E821F3
+P 5850 3100
+F 0 "K?" V 5800 3100 50  0000 C CNN
+F 1 "CONN_3" V 5900 3100 40  0000 C CNN
+F 2 "" H 5850 3100 60  0000 C CNN
+F 3 "" H 5850 3100 60  0000 C CNN
+	1    5850 3100
+	1    0    0    -1
+$EndComp
 $EndSCHEMATC

Commit message: Elec ?
Parts:
- gave numbers to parts that had none: 1
Changed lines of the file:
@@
 OUT
 $Comp
-L CONN_3 K?
+L CONN_3 K8
 U 1 1 55E821F3
 P 5850 3100
-F 0 "K?" V 5800 3100 50  0000 C CNN
+AR Path="/55E6307C/55E6315E/55E821F3" Ref="K8"  Part="1"
+AR Path="/55E7381B/55E6315E/55E821F3" Ref="K2"  Part="1"
+AR Path="/55E7381C/55E6315E/55E821F3" Ref="K4"  Part="1"
+AR Path="/55E7381D/55E6315E/55E821F3" Ref="K6"  Part="1"
+F 0 "K8" V 5800 3100 50  0000 C CNN
 F 1 "CONN_3" V 5900 3100 40  0000 C CNN
 F 2 "" H 5850 3100 60  0000 C CNN
