File: elec/teensy_shield/joint.sch (KiCad schematic (older format))
At the start: 0 parts

Commit message: Completed new board schematics.
Changed lines of the file:
@@
 LIBS:contrib
 LIBS:valves
+LIBS:arduino_shieldsNCL
+LIBS:teensy
+LIBS:pololu
+LIBS:teensy_shield-cache
 EELAYER 24 0
 EELAYER END
 $Descr A4 11693 8268
 encoding utf-8
-Sheet 4 26
+Sheet 4 34
 Title ""
 Date ""
@@
 Text HLabel 4800 1900 0    60   Input ~ 0
 Vin_pow
-Text HLabel 4300 3550 0    60   Input ~ 0
+Text HLabel 4250 3550 0    60   Input ~ 0
 PWM
 Text HLabel 4800 3650 0    60   Input ~ 0
@@
 F5 "EN" I L 4800 2100 60
 $EndSheet
-$Sheet
-S 4800 3050 600  700
-U 55E6553A
-F0 "motor_driver" 50
-F1 "motor_driver.sch" 50
-F2 "Vin" I L 4800 3250 60
-F3 "GND" I L 4800 3150 60
-F4 "M2" O R 5400 3250 60
-F5 "nEN" I L 4800 3350 60
-F6 "nFAULT" I L 4800 3450 60
-F7 "M1" O R 5400 3350 60
-F8 "DIR" I L 4800 3650 60
-F9 "PWM" I L 4800 3550 60
-$EndSheet
-Wire Wire Line
-	5400 3350 5700 3350
-Wire Wire Line
-	5700 3350 5700 4050
-Wire Wire Line
-	5700 4050 5500 4050
-Wire Wire Line
-	5500 4150 6250 4150
-Wire Wire Line
-	6250 4150 6250 3350
-Wire Wire Line
-	6250 3350 6350 3350
 Wire Wire Line
 	6350 3250 5400 3250
-Text Label 4800 3250 2    60   ~ 0
-Vmot
-Text Label 4800 2000 2    60   ~ 0
-Vmot
 Text HLabel 4800 2100 0    60   Input ~ 0
 EN
 Wire Wire Line
-	4300 3550 4400 3550
+	4250 3550 4350 3550
 Wire Wire Line
-	4400 3550 4800 3550
+	4350 3550 4800 3550
 Wire Wire Line
-	4800 2700 4400 2700
+	4800 2700 4350 2700
 Wire Wire Line
-	4400 2700 4400 3550
-Connection ~ 4400 3550
-Text Label 4800 2600 2    60   ~ 0
-Vmot
+	4350 2700 4350 3550
+Connection ~ 4350 3550
 Text Label 3550 3000 0    60   ~ 0
 GND
@@
 GND
 Wire Wire Line
-	4800 4900 4200 4900
+	4100 4900 4200 4900
 Wire Wire Line
-	4200 4900 4100 4900
+	4200 4900 4800 4900
 Wire Wire Line
 	4800 4150 4200 4150
@@
 	4200 4150 4200 4900
 Connection ~ 4200 4900
+$Sheet
+S 4800 3050 600  700
+U 55E6553A
+F0 "motor_driver" 50
+F1 "motor_driver.sch" 50
+F2 "Vin" I L 4800 3250 60
+F3 "GND" I L 4800 3150 60
+F4 "M2" O R 5400 3250 60
+F5 "nEN" I L 4800 3350 60
+F6 "nFAULT" I L 4800 3450 60
+F7 "M1" O R 5400 3350 60
+F8 "DIR" I L 4800 3650 60
+F9 "PWM" I L 4800 3550 60
+$EndSheet
+Text Label 4800 2000 2    60   ~ 0
+Vpow_IP+
+Text Label 5500 4050 0    60   ~ 0
+Vpow_IP+
+Text Label 5500 4150 0    60   ~ 0
+Vpow_IP-
+Text Label 4800 2600 2    60   ~ 0
+Vpow_IP-
+Text Label 4800 3250 2    60   ~ 0
+Vpow_IP-
+Wire Wire Line
+	5400 3350 6350 3350
 $EndSCHEMATC

Commit message: Elec ?
Changed lines of the file:
@@
 $Descr A4 11693 8268
 encoding utf-8
-Sheet 4 34
+Sheet 18 34
 Title ""
 Date ""
@@
 F3 "GND" I L 4800 4050 60
 F4 "OUT" I L 4800 4250 60
-F5 "nFAULT" I L 4800 4350 60
-F6 "IP+" I R 5500 4050 60
-F7 "IP-" I R 5500 4150 60
+F5 "IP+" I R 5500 4050 60
+F6 "IP-" I R 5500 4150 60
 $EndSheet
 $Sheet
@@
 F0 "motor" 50
 F1 "motor.sch" 50
-F2 "GND" I L 6350 3150 60
-F3 "M+" I L 6350 3350 60
-F4 "M-" I L 6350 3250 60
+F2 "M+" I L 6350 3350 60
+F3 "M-" I L 6350 3250 60
 $EndSheet
 $Sheet
@@
 EN
 Wire Wire Line
-	4250 3550 4350 3550
-Wire Wire Line
-	4350 3550 4800 3550
+	4250 3550 4800 3550
 Wire Wire Line
 	4800 2700 4350 2700
@@
 GND
 Wire Wire Line
-	4100 4900 4200 4900
-Wire Wire Line
-	4200 4900 4800 4900
+	4100 4900 4800 4900
 Wire Wire Line
 	4800 4150 4200 4150
@@
 F3 "GND" I L 4800 3150 60
 F4 "M2" O R 5400 3250 60
-F5 "nEN" I L 4800 3350 60
-F6 "nFAULT" I L 4800 3450 60
-F7 "M1" O R 5400 3350 60
-F8 "DIR" I L 4800 3650 60
-F9 "PWM" I L 4800 3550 60
+F5 "M1" O R 5400 3350 60
+F6 "DIR" I L 4800 3650 60
+F7 "PWM" I L 4800 3550 60
 $EndSheet
 Text Label 4800 2000 2    60   ~ 0
